File: d-lev-main/AFE.kicad_sch (KiCad schematic)
At the start: 2 parts, among them J7 SM07B-SRSS-TB(LF)(SN), X3 A07SR07SR30K152A

Commit message: Many changes
Reorganized libraries to share between projects
Set up JLC 2- and 4- layer design rules
Finished copying over most of the schematic (excluding I/O board)
Parts:
- removed J7: SM07B-SRSS-TB(LF)(SN), symbol Connector_Generic:Conn_01x07
- removed X3: A07SR07SR30K152A, symbol assorted:BOM ITEM
Other:
- note removed: "Mates with:"
- note removed: "http://www.helloxkb.com/Home/Goods/goodsInfo/id/368.html"
Changed lines of the file:
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@@
 (kicad_sch (version 20230121) (generator eeschema)
   (paper "A4")
-  (wire (pts (xy 144.78 92.075) (xy 149.225 92.075))
-    (stroke (width 0) (type default))
-  )
-  (wire (pts (xy 149.225 99.695) (xy 144.78 99.695))
-    (stroke (width 0) (type default))
-  )
-  (wire (pts (xy 144.78 97.155) (xy 149.225 97.155))
-    (stroke (width 0) (type default))
-  )
-  (wire (pts (xy 149.225 104.775) (xy 144.78 104.775))
-    (stroke (width 0) (type default))
-  )
-  (wire (pts (xy 144.78 89.535) (xy 149.225 89.535))
-    (stroke (width 0) (type default))
-  )
-  (wire (pts (xy 144.78 102.235) (xy 149.225 102.235))
-    (stroke (width 0) (type default))
-  )
-  (wire (pts (xy 149.225 94.615) (xy 144.78 94.615))
-    (stroke (width 0) (type default))
-  )
-  (text "Mates with:" (at 170.815 108.585 0)
-    (effects (font (size 1.27 1.27)) (justify left bottom))
-  )
-  (text "http://www.helloxkb.com/Home/Goods/goodsInfo/id/368.html"
-    (at 162.56 88.9 0)
-    (effects (font (size 1.27 1.27)) (justify left bottom))
-  )
-  (hierarchical_label "zero_i" (shape input) (at 144.78 94.615 180) (fields_autoplaced)
-    (effects (font (size 1.27 1.27)) (justify right))
-  )
-  (hierarchical_label "sq_o" (shape output) (at 144.78 99.695 180) (fields_autoplaced)
-    (effects (font (size 1.27 1.27)) (justify right))
-  )
-  (hierarchical_label "quad_i" (shape input) (at 144.78 89.535 180) (fields_autoplaced)
-    (effects (font (size 1.27 1.27)) (justify right))
-  )
-  (hierarchical_label "afe_gnd" (shape input) (at 144.78 92.075 180) (fields_autoplaced)
-    (effects (font (size 1.27 1.27)) (justify right))
-  )
-  (hierarchical_label "afe_gnd" (shape input) (at 144.78 97.155 180) (fields_autoplaced)
-    (effects (font (size 1.27 1.27)) (justify right))
-  )
-  (hierarchical_label "afe_power" (shape input) (at 144.78 104.775 180) (fields_autoplaced)
-    (effects (font (size 1.27 1.27)) (justify right))
-  )
-  (hierarchical_label "afe_gnd" (shape input) (at 144.78 102.235 180) (fields_autoplaced)
-    (effects (font (size 1.27 1.27)) (justify right))
-  )
-  (symbol (lib_id "assorted:BOM ITEM") (at 175.895 111.76 0) (unit 1)
-    (in_bom yes) (on_board no) (dnp no)
-    (property "Reference" "X3" (at 175.895 111.76 0)
-      (effects (font (size 1.27 1.27)) hide)
-    )
-    (property "Value" "A07SR07SR30K152A" (at 165.735 111.76 0)
-      (effects (font (size 1.27 1.27)) (justify left))
-    )
-    (property "Footprint" "" (at 175.895 111.76 0)
-      (effects (font (size 1.27 1.27)) hide)
-    )
-    (property "Datasheet" "https://gam-gec.com/wp-content/uploads/2018/10/GAM-011.pdf" (at 175.895 111.76 0)
-      (effects (font (size 1.27 1.27)) hide)
-    )
-    (instances
-      (project "dlev-mini"
-        (path "/eb5e8bfd-9871-4528-bf57-58851bf63907/94220e47-26ce-4172-b51a-d5169ade8ea4"
-          (reference "X3") (unit 1)
-        )
-        (path "/eb5e8bfd-9871-4528-bf57-58851bf63907/e6848102-2669-4daa-a892-b8781bc3a056"
-          (reference "X2") (unit 1)
-        )
-      )
-    )
-  )
-  (symbol (lib_id "Connector_Generic:Conn_01x07") (at 154.305 97.155 0) (unit 1)
-    (in_bom yes) (on_board yes) (dnp no) (fields_autoplaced)
-    (property "Reference" "J7" (at 156.845 95.8849 0)
-      (effects (font (size 1.27 1.27)) (justify left))
-    )
-    (property "Value" "SM07B-SRSS-TB(LF)(SN)" (at 156.845 98.4249 0)
-      (effects (font (size 1.27 1.27)) (justify left))
-    )
-    (property "Footprint" "" (at 154.305 97.155 0)
-      (effects (font (size 1.27 1.27)) hide)
-    )
-    (property "Datasheet" "https://www.jst-mfg.com/product/pdf/eng/eSH.pdf" (at 154.305 97.155 0)
-      (effects (font (size 1.27 1.27)) hide)
-    )
-    (pin "1")
-    (pin "2")
-    (pin "3")
-    (pin "4")
-    (pin "5")
-    (pin "6")
-    (pin "7")
-    (instances
-      (project "dlev-mini"
-        (path "/eb5e8bfd-9871-4528-bf57-58851bf63907/94220e47-26ce-4172-b51a-d5169ade8ea4"
-          (reference "J7") (unit 1)
-        )
-        (path "/eb5e8bfd-9871-4528-bf57-58851bf63907/e6848102-2669-4daa-a892-b8781bc3a056"
-          (reference "J6") (unit 1)
-        )
-      )
-    )
-  )
 )
