File: d-lev-main/dlev-mini.kicad_pcb (KiCad board)
At the start: 4 copper layers, 208.9 x 161.9 mm, 25 parts, among them J1 IO_BOARD, J2 Tag-Connect TC2030-NL, J3 S8B-PH-SM4-TB, J4 S8B-PH-SM4-TB, J6 S6B-PH-SM4-TB, Q1 MMBT3904, Q2 MMBT3904, SW1 RotaryEncoder_Switch, SW2 RotaryEncoder_Switch, SW3 RotaryEncoder_Switch, SW4 RotaryEncoder_Switch, SW5 RotaryEncoder_Switch, SW6 RotaryEncoder_Switch, SW7 RotaryEncoder_Switch, SW8 RotaryEncoder_Switch, U2 AMS1117-3.3, U3 AC608, U4 25LCxxx

Commit message: Level shifters and rearrange encoders
* WIP: use net buses more effectively to organize encoder signals
* Add application note for level shifters
* Add level shifters for UART, change MIDI level shifter BJT to FET
* Add MIDI_HI pull-up on d-lev-io board
* Add/change some footprints
Parts:
- removed Q1: MMBT3904, Package_TO_SOT_SMD:SOT-23
- removed U4: 25LCxxx, Package_SO:SOIC-8W_5.3x5.3mm_P1.27mm
- added C1: .01u, Capacitor_SMD:C_0805_2012Metric_Pad1.18x1.45mm_HandSolder, F.Cu at (22.3, 20.7)
- added C10: .1u, Capacitor_SMD:C_0805_2012Metric_Pad1.18x1.45mm_HandSolder, F.Cu at (27.7, 4.55)
- added C11: .01u, Capacitor_SMD:C_0805_2012Metric_Pad1.18x1.45mm_HandSolder, F.Cu at (16.2, 10.0)
- added C12: .01u, Capacitor_SMD:C_0805_2012Metric_Pad1.18x1.45mm_HandSolder, F.Cu at (1.91, 20.7)
- added C13: .01u, Capacitor_SMD:C_0805_2012Metric_Pad1.18x1.45mm_HandSolder, F.Cu at (1.91, 23.7)
- added C14: .01u, Capacitor_SMD:C_0805_2012Metric_Pad1.18x1.45mm_HandSolder, F.Cu at (15.5, 20.7)
- added C15: .01u, Capacitor_SMD:C_0805_2012Metric_Pad1.18x1.45mm_HandSolder, F.Cu at (15.5, 23.7)
- added C16: .01u, Capacitor_SMD:C_0805_2012Metric_Pad1.18x1.45mm_HandSolder, F.Cu at (15.5, 31.7)
- added C17: .01u, Capacitor_SMD:C_0805_2012Metric_Pad1.18x1.45mm_HandSolder, F.Cu at (15.5, 34.7)
- added C18: .01u, Capacitor_SMD:C_0805_2012Metric_Pad1.18x1.45mm_HandSolder, F.Cu at (22.3, 31.7)
- added C19: .01u, Capacitor_SMD:C_0805_2012Metric_Pad1.18x1.45mm_HandSolder, F.Cu at (22.3, 34.7)
- added C2: .01u, Capacitor_SMD:C_0805_2012Metric_Pad1.18x1.45mm_HandSolder, F.Cu at (22.3, 23.7)
- added C20: .01u, Capacitor_SMD:C_0805_2012Metric_Pad1.18x1.45mm_HandSolder, F.Cu at (8.71, 20.7)
- added C21: .01u, Capacitor_SMD:C_0805_2012Metric_Pad1.18x1.45mm_HandSolder, F.Cu at (8.71, 23.7)
- added C3: .01u, Capacitor_SMD:C_0805_2012Metric_Pad1.18x1.45mm_HandSolder, F.Cu at (1.91, 31.7)
- added C4: .01u, Capacitor_SMD:C_0805_2012Metric_Pad1.18x1.45mm_HandSolder, F.Cu at (1.91, 34.7)
- added C5: .01u, Capacitor_SMD:C_0805_2012Metric_Pad1.18x1.45mm_HandSolder, F.Cu at (8.71, 31.7)
- added C6: .01u, Capacitor_SMD:C_0805_2012Metric_Pad1.18x1.45mm_HandSolder, F.Cu at (8.71, 34.7)
- added C7: 22u, Capacitor_SMD:C_0805_2012Metric_Pad1.18x1.45mm_HandSolder, F.Cu at (16.2, 1.00)
- added C8: 22u, Capacitor_SMD:C_0805_2012Metric_Pad1.18x1.45mm_HandSolder, F.Cu at (16.2, 4.01)
- added C9: .01u, Capacitor_SMD:C_0805_2012Metric_Pad1.18x1.45mm_HandSolder, F.Cu at (16.2, 7.03)
- added JP1: LCD_VSEL, Jumper:SolderJumper-3_P1.3mm_Bridged2Bar12_RoundedPad1.0x1.5mm_NumberLabels, F.Cu at (28.1, 1.27)
- added Q3: BSS138, Package_TO_SOT_SMD:SOT-23, F.Cu at (178.2, -17.9)
- added Q4: BSS138, Package_TO_SOT_SMD:SOT-23, F.Cu at (178.2, -13.4)
- added Q5: BSS138, Package_TO_SOT_SMD:SOT-23, F.Cu at (178.2, -8.96)
- added R10: 470, Resistor_SMD:R_0805_2012Metric_Pad1.20x1.40mm_HandSolder, F.Cu at (1.88, 6.88)
- added R11: 470, Resistor_SMD:R_0805_2012Metric_Pad1.20x1.40mm_HandSolder, F.Cu at (1.88, 9.82)
- added R12: 470, Resistor_SMD:R_0805_2012Metric_Pad1.20x1.40mm_HandSolder, F.Cu at (1.88, 12.8)
- added R14: 10k, Resistor_SMD:R_0805_2012Metric_Pad1.20x1.40mm_HandSolder, F.Cu at (1.88, 15.7)
- added R15: 10k, Resistor_SMD:R_0805_2012Metric_Pad1.20x1.40mm_HandSolder, F.Cu at (6.62, 0.97)
- added R16: 10k, Resistor_SMD:R_0805_2012Metric_Pad1.20x1.40mm_HandSolder, F.Cu at (6.62, 3.92)
- added R17: 10k, Resistor_SMD:R_0805_2012Metric_Pad1.20x1.40mm_HandSolder, F.Cu at (6.62, 6.88)
- added R18: 10k, Resistor_SMD:R_0805_2012Metric_Pad1.20x1.40mm_HandSolder, F.Cu at (6.62, 9.82)
- added R19: 10k, Resistor_SMD:R_0805_2012Metric_Pad1.20x1.40mm_HandSolder, F.Cu at (6.62, 12.8)
- added R20: 10k, Resistor_SMD:R_0805_2012Metric_Pad1.20x1.40mm_HandSolder, F.Cu at (6.62, 15.7)
- added R21: 10k, Resistor_SMD:R_0805_2012Metric_Pad1.20x1.40mm_HandSolder, F.Cu at (11.4, 0.97)
- added R22: 1k, Resistor_SMD:R_0805_2012Metric_Pad1.20x1.40mm_HandSolder, F.Cu at (11.4, 3.92)
- added R23: 1k, Resistor_SMD:R_0805_2012Metric_Pad1.20x1.40mm_HandSolder, F.Cu at (11.4, 6.88)
- added R24: 220, Resistor_SMD:R_0805_2012Metric_Pad1.20x1.40mm_HandSolder, F.Cu at (11.4, 9.82)
- added R3: 10k, Resistor_SMD:R_0805_2012Metric_Pad1.20x1.40mm_HandSolder, F.Cu at (1.88, 0.97)
- added R5: 1k, Resistor_SMD:R_0805_2012Metric_Pad1.20x1.40mm_HandSolder, F.Cu at (22.9, 0.97)
- added R6: 22, Resistor_SMD:R_0805_2012Metric_Pad1.20x1.40mm_HandSolder, F.Cu at (22.9, 3.92)
- added R7: 1k, Resistor_SMD:R_0805_2012Metric_Pad1.20x1.40mm_HandSolder, F.Cu at (22.9, 6.88)
- added R8: 1k, Resistor_SMD:R_0805_2012Metric_Pad1.20x1.40mm_HandSolder, F.Cu at (22.9, 9.82)
- added R9: 470, Resistor_SMD:R_0805_2012Metric_Pad1.20x1.40mm_HandSolder, F.Cu at (1.88, 3.92)
- added RN1: 10k, Resistor_SMD:R_Array_Concave_4x0603, F.Cu at (22.3, 26.7)
- added RN2: 10k, Resistor_SMD:R_Array_Concave_4x0603, F.Cu at (1.88, 37.7)
- added RN3: 10k, Resistor_SMD:R_Array_Concave_4x0603, F.Cu at (8.69, 37.7)
- added RN4: 10k, Resistor_SMD:R_Array_Concave_4x0603, F.Cu at (1.88, 26.7)
- added RN5: 10k, Resistor_SMD:R_Array_Concave_4x0603, F.Cu at (15.5, 26.7)
- added RN6: 10k, Resistor_SMD:R_Array_Concave_4x0603, F.Cu at (15.5, 37.7)
- added RN7: 10k, Resistor_SMD:R_Array_Concave_4x0603, F.Cu at (22.3, 37.7)
- added RN8: 10k, Resistor_SMD:R_Array_Concave_4x0603, F.Cu at (8.69, 26.7)
- added RV1: 10K, Potentiometer_SMD:Potentiometer_Bourns_3269P_Horizontal, F.Cu at (22.9, 12.8)
- added U1: 25LCxxx, Package_SO:SOIC-8W_5.3x5.3mm_P1.27mm, F.Cu at (185.9, -16.6)
- R1, R2: value 5.1k -> 10k
- moved SW8 118.6 mm to (38.9, 36.4)
Connections:
- net /Encoders/S0 renamed /Encoders/SingleEncoder3/OUT.S
- net /Encoders/S1 renamed /Encoders/SingleEncoder4/OUT.S
- net /Encoders/S2 renamed /Encoders/SingleEncoder5/OUT.S
- net /Encoders/S3 renamed /Encoders/SingleEncoder6/OUT.S
- net /Encoders/S4 renamed /Encoders/SingleEncoder7/OUT.S
- net /Encoders/S5 renamed /Encoders/SingleEncoder8/OUT.S
- net /Encoders/S6 renamed /Encoders/SingleEncoder9/OUT.S
- net /Encoders/S7 renamed /Encoders/SingleEncoder10/OUT.S
- net /FPGA/lcd_data0 renamed /FPGA/lcd.data0
- net /FPGA/lcd_data1 renamed /FPGA/lcd.data1
- net /FPGA/lcd_data2 renamed /FPGA/lcd.data2
- net /FPGA/lcd_data3 renamed /FPGA/lcd.data3
- DS2 pad 6: /FPGA/lcd.rs -> /FPGA/lcd.e
- J1 pad 11: unconnected-(J1-Pin_11-Pad11) -> mute_led
- J1 pad 12: unconnected-(J1-Pin_12-Pad12) -> GND
- J1 pad 3: uart_tx -> uart_tx_5v
- J1 pad 4: uart_rx -> uart_rx_5v
- J1 pad 5: midi_out -> midi_out_lo
- R1 pad 1: GND -> /FPGA/mem_spi.cs
- R1 pad 2: Net-(J4-PadA5) -> GND
- R2 pad 1: GND -> Net-(U1-~{WP})
- R2 pad 2: Net-(J4-PadB5) -> +3V3
- SW1 pad A: /Encoders/A0 -> /Encoders/SingleEncoder3/A1
- SW1 pad B: /Encoders/B0 -> /Encoders/SingleEncoder3/B1
- SW2 pad A: /Encoders/A1 -> /Encoders/SingleEncoder4/A1
- SW2 pad B: /Encoders/B1 -> /Encoders/SingleEncoder4/B1
- SW3 pad A: /Encoders/A2 -> /Encoders/SingleEncoder5/A1
- SW3 pad B: /Encoders/B2 -> /Encoders/SingleEncoder5/B1
- SW4 pad A: /Encoders/A3 -> /Encoders/SingleEncoder6/A1
- SW4 pad B: /Encoders/B3 -> /Encoders/SingleEncoder6/B1
- SW5 pad A: /Encoders/A4 -> /Encoders/SingleEncoder7/A1
- SW5 pad B: /Encoders/B4 -> /Encoders/SingleEncoder7/B1
- SW6 pad A: /Encoders/A5 -> /Encoders/SingleEncoder8/A1
- SW6 pad B: /Encoders/B5 -> /Encoders/SingleEncoder8/B1
- SW7 pad A: /Encoders/A6 -> /Encoders/SingleEncoder9/A1
- SW7 pad B: /Encoders/B6 -> /Encoders/SingleEncoder9/B1
- SW8 pad A: /Encoders/A7 -> /Encoders/SingleEncoder10/A1
- SW8 pad B: /Encoders/B7 -> /Encoders/SingleEncoder10/B1
- U3 pad 88: unconnected-(U3-LVDS_TX2_N-Pad88) -> /FPGA/enc_s0

Commit message: more encoder bus mangling
Parts:
- moved SW5 185.9 mm to (74.6, 12.4)
- moved SW4 178.3 mm to (74.6, -12.4)
- moved SW2 162.5 mm to (48.2, 12.4)
- moved SW8 160.4 mm to (180.3, 111.9)
- moved SW3 140.8 mm to (74.6, 37.2)
- moved SW7 117.3 mm to (48.2, -12.4)
- moved C16 101.8 mm to (113.2, 2.83)
- moved C17 101.8 mm to (113.2, 5.84)
- moved RN6 101.3 mm to (112.9, 9.76)
- moved C1 100.4 mm to (113.2, -22.0)
- moved C2 100.4 mm to (113.2, -19.0)
- moved RN1 99.7 mm to (112.9, -15.0)
- moved C12 95.0 mm to (86.8, -22.0)
- moved C13 95.0 mm to (86.8, -19.0)
- moved RN4 94.3 mm to (86.5, -15.0)
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Connections:
- net /Encoders/SingleEncoder10/A1 renamed /Encoders/Encoder0/A1
- net /Encoders/SingleEncoder10/B1 renamed /Encoders/Encoder0/B1
- net /Encoders/SingleEncoder10/OUT.A renamed /Encoders/Encoder0/OUT.A
- net /Encoders/SingleEncoder10/OUT.B renamed /Encoders/Encoder0/OUT.B
- net /Encoders/SingleEncoder10/OUT.S renamed /Encoders/Encoder0/OUT.S
- net /Encoders/SingleEncoder3/OUT.A renamed /Encoders/Encoder2/OUT.A
- net /Encoders/SingleEncoder3/OUT.B renamed /Encoders/Encoder2/OUT.B
- net /Encoders/SingleEncoder3/OUT.S renamed /Encoders/Encoder1/OUT.S
- net /Encoders/SingleEncoder4/OUT.A renamed /Encoders/Encoder1/OUT.A
- net /Encoders/SingleEncoder4/OUT.B renamed /Encoders/Encoder1/OUT.B
- net /Encoders/SingleEncoder4/OUT.S renamed /Encoders/Encoder2/OUT.S
- net /Encoders/SingleEncoder5/A1 renamed /Encoders/Encoder3/A1
- net /Encoders/SingleEncoder5/B1 renamed /Encoders/Encoder3/B1
- net /Encoders/SingleEncoder5/OUT.A renamed /Encoders/Encoder3/OUT.A
- net /Encoders/SingleEncoder5/OUT.B renamed /Encoders/Encoder3/OUT.B
- net /Encoders/SingleEncoder5/OUT.S renamed /Encoders/Encoder3/OUT.S
- net /Encoders/SingleEncoder6/A1 renamed /Encoders/Encoder5/A1
- net /Encoders/SingleEncoder6/B1 renamed /Encoders/Encoder5/B1
- net /Encoders/SingleEncoder6/OUT.A renamed /Encoders/Encoder5/OUT.A
- net /Encoders/SingleEncoder6/OUT.B renamed /Encoders/Encoder5/OUT.B
- net /Encoders/SingleEncoder6/OUT.S renamed /Encoders/Encoder5/OUT.S
- net /Encoders/SingleEncoder7/A1 renamed /Encoders/Encoder6/A1
- net /Encoders/SingleEncoder7/B1 renamed /Encoders/Encoder6/B1
- net /Encoders/SingleEncoder7/OUT.A renamed /Encoders/Encoder6/OUT.A
- net /Encoders/SingleEncoder7/OUT.B renamed /Encoders/Encoder6/OUT.B
- net /Encoders/SingleEncoder7/OUT.S renamed /Encoders/Encoder6/OUT.S
- net /Encoders/SingleEncoder8/A1 renamed /Encoders/Encoder4/A1
- net /Encoders/SingleEncoder8/B1 renamed /Encoders/Encoder4/B1
- net /Encoders/SingleEncoder8/OUT.A renamed /Encoders/Encoder4/OUT.A
- net /Encoders/SingleEncoder8/OUT.B renamed /Encoders/Encoder4/OUT.B
- net /Encoders/SingleEncoder8/OUT.S renamed /Encoders/Encoder4/OUT.S
- net /Encoders/SingleEncoder9/A1 renamed /Encoders/Encoder7/A1
- net /Encoders/SingleEncoder9/B1 renamed /Encoders/Encoder7/B1
- net /Encoders/SingleEncoder9/OUT.A renamed /Encoders/Encoder7/OUT.A
- net /Encoders/SingleEncoder9/OUT.B renamed /Encoders/Encoder7/OUT.B
- net /Encoders/SingleEncoder9/OUT.S renamed /Encoders/Encoder7/OUT.S
- net /FPGA/enc_s0 renamed /Encoders/Encoder0/enc.a
- RN1 pad 1: /Encoders/SingleEncoder4/B1 -> /Encoders/Encoder1/B1
- RN1 pad 2: /Encoders/SingleEncoder4/A1 -> /Encoders/Encoder1/A1
- RN1 pad 3: /Encoders/SingleEncoder4/A1 -> /Encoders/Encoder1/A1
- RN1 pad 4: /Encoders/SingleEncoder4/B1 -> /Encoders/Encoder1/B1
- RN2 pad 1: /Encoders/SingleEncoder3/B1 -> /Encoders/Encoder2/B1
- RN2 pad 2: /Encoders/SingleEncoder3/A1 -> /Encoders/Encoder2/A1
- RN2 pad 3: /Encoders/SingleEncoder3/A1 -> /Encoders/Encoder2/A1
- RN2 pad 4: /Encoders/SingleEncoder3/B1 -> /Encoders/Encoder2/B1
- SW1 pad A: /Encoders/SingleEncoder3/A1 -> /Encoders/Encoder1/A1
- SW1 pad B: /Encoders/SingleEncoder3/B1 -> /Encoders/Encoder1/B1
- SW2 pad A: /Encoders/SingleEncoder4/A1 -> /Encoders/Encoder2/A1
- SW2 pad B: /Encoders/SingleEncoder4/B1 -> /Encoders/Encoder2/B1
- U3 pad 86: unconnected-(U3-LVDS_TX1_N-Pad86) -> /Encoders/Encoder0/enc.s
- U3 pad 87: unconnected-(U3-LVDS_TX1_P-Pad87) -> /Encoders/Encoder0/enc.b
Routing:
- net /Encoders/Encoder0/enc.s: track 0.00 -> 1.91 mm
Other:
- board size 208.9 x 161.9 mm -> 330.4 x 275 mm

Commit message: Small changes to 3D models and footprints; fixed bus routing of encoder signals
Parts:
- removed J6: S6B-PH-SM4-TB, d-lev:JST_PH_S6B-PH-SM4-TB_1x06-1MP_P2.00mm_Horizontal
- added J5: Conn_01x06_MountingPin, d-lev:JST_PH_S6B-PH-SM4-TB_1x06-1MP_P2.00mm_Horizontal, F.Cu at (83.9, 111.8)
- DS2: footprint d-lev:ERM2004-1 -> d-lev:ERM2004-0
- H1, H3, H4: value MountingHole -> MountingHole_Pad
- J1: value IO_BOARD -> Conn_01x12_MountingPin
- RV1: footprint Potentiometer_SMD:Potentiometer_Bourns_3269P_Horizontal -> Potentiometer_SMD:Potentiometer_Bourns_TC33X_Vertical
- SW1, SW2, SW3, SW4, SW5, SW6, SW7, SW8: footprint d-lev:PEC11S9215FS0015 -> d-lev:PEC11S-929K
- moved U1 180.7 mm to (86.3, 134.2)
- moved R1 179.4 mm to (69.2, 118.9)
- moved H3 171.6 mm to (70.5, 91.0)
- moved Q3 166.9 mm to (83.5, 119.6)
- moved Q4 166.9 mm to (83.5, 124.1)
- moved Q5 166.9 mm to (83.5, 128.5)
- moved C12 166.6 mm to (119.9, 141.3)
- moved C13 166.6 mm to (119.9, 144.3)
- moved RN4 166.6 mm to (119.5, 148.2)
- moved C18 162.9 mm to (146.3, 116.5)
- moved C19 162.9 mm to (146.3, 119.5)
- moved RN7 162.9 mm to (145.9, 123.4)
- moved SW4 162.9 mm to (160.5, 126.0)
- moved H1 157.8 mm to (49.7, 91.0)
- moved H2 152.6 mm to (60.1, 91.0)
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Connections:
- net /Encoders/Encoder0/A1 renamed /encoder6/A1
- net /Encoders/Encoder0/B1 renamed /encoder6/B1
- net /Encoders/Encoder0/OUT.A renamed enc_8.a
- net /Encoders/Encoder0/OUT.B renamed enc_8.b
- net /Encoders/Encoder0/OUT.S renamed enc_8.s
- net /Encoders/Encoder1/A1 renamed /encoder1/A1
- net /Encoders/Encoder1/B1 renamed /encoder1/B1
- net /Encoders/Encoder1/OUT.A renamed enc_2.a
- net /Encoders/Encoder1/OUT.B renamed enc_2.b
- net /Encoders/Encoder1/OUT.S renamed enc_2.s
- net /Encoders/Encoder2/OUT.A renamed enc_3.a
- net /Encoders/Encoder2/OUT.B renamed enc_3.b
- net /Encoders/Encoder2/OUT.S renamed enc_1.s
- net /Encoders/Encoder3/OUT.A renamed enc_4.a
- net /Encoders/Encoder3/OUT.B renamed enc_4.b
- net /Encoders/Encoder3/OUT.S renamed enc_3.s
- net /Encoders/Encoder4/OUT.A renamed enc_7.a
- net /Encoders/Encoder4/OUT.B renamed enc_7.b
- net /Encoders/Encoder4/OUT.S renamed enc_5.s
- net /Encoders/Encoder5/OUT.A renamed enc_6.a
- net /Encoders/Encoder5/OUT.B renamed enc_6.b
- net /Encoders/Encoder5/OUT.S renamed enc_4.s
- net /Encoders/Encoder6/OUT.A renamed enc_5.a
- net /Encoders/Encoder6/OUT.B renamed enc_5.b
- net /Encoders/Encoder6/OUT.S renamed enc_6.s
- net /Encoders/Encoder7/OUT.A renamed enc_1.a
- net /Encoders/Encoder7/OUT.B renamed enc_1.b
- net /Encoders/Encoder7/OUT.S renamed enc_7.s
- H1 pad 1: (no net) -> GND
- H3 pad 1: (no net) -> GND
- H4 pad 1: (no net) -> GND
- J1 pad MP: (no net) -> unconnected-(J1-MountPin-PadMP)
- J3 pad MP: (no net) -> unconnected-(J3-MountPin-PadMP)
- J4 pad MP: (no net) -> unconnected-(J4-MountPin-PadMP)
- RN2 pad 1: /Encoders/Encoder2/B1 -> /encoder2/B1
- RN2 pad 2: /Encoders/Encoder2/A1 -> /encoder2/A1
- RN2 pad 3: /Encoders/Encoder2/A1 -> /encoder2/A1
- RN2 pad 4: /Encoders/Encoder2/B1 -> /encoder2/B1
- RN3 pad 1: /Encoders/Encoder3/B1 -> /encoder3/B1
- RN3 pad 2: /Encoders/Encoder3/A1 -> /encoder3/A1
- RN3 pad 3: /Encoders/Encoder3/A1 -> /encoder3/A1
- RN3 pad 4: /Encoders/Encoder3/B1 -> /encoder3/B1
- RN4 pad 1: /Encoders/Encoder5/B1 -> /encoder4/B1
- RN4 pad 2: /Encoders/Encoder5/A1 -> /encoder4/A1
- RN4 pad 3: /Encoders/Encoder5/A1 -> /encoder4/A1
- RN4 pad 4: /Encoders/Encoder5/B1 -> /encoder4/B1
- RN5 pad 1: /Encoders/Encoder6/B1 -> /encoder7/B1
- RN5 pad 2: /Encoders/Encoder6/A1 -> /encoder7/A1
- RN5 pad 3: /Encoders/Encoder6/A1 -> /encoder7/A1
- RN5 pad 4: /Encoders/Encoder6/B1 -> /encoder7/B1
- RN6 pad 1: /Encoders/Encoder4/B1 -> /encoder5/B1
- RN6 pad 2: /Encoders/Encoder4/A1 -> /encoder5/A1
- RN6 pad 3: /Encoders/Encoder4/A1 -> /encoder5/A1
- RN6 pad 4: /Encoders/Encoder4/B1 -> /encoder5/B1
- RN7 pad 1: /Encoders/Encoder7/B1 -> /encoder/B1
- RN7 pad 2: /Encoders/Encoder7/A1 -> /encoder/A1
- RN7 pad 3: /Encoders/Encoder7/A1 -> /encoder/A1
- RN7 pad 4: /Encoders/Encoder7/B1 -> /encoder/B1
- SW1 pad MP1: (no net) -> unconnected-(SW1-PadMP1)
- SW1 pad MP2: (no net) -> unconnected-(SW1-PadMP2)
- SW1 pad MP3: (no net) -> unconnected-(SW1-PadMP3)
- SW1 pad MP4: (no net) -> unconnected-(SW1-PadMP4)
- SW1 pad MP5: (no net) -> unconnected-(SW1-PadMP5)
- SW1 pad MP6: (no net) -> unconnected-(SW1-PadMP6)
- SW2 pad A: /Encoders/Encoder2/A1 -> /encoder/A1
- SW2 pad B: /Encoders/Encoder2/B1 -> /encoder/B1
- SW2 pad MP1: (no net) -> unconnected-(SW2-PadMP1)
- SW2 pad MP2: (no net) -> unconnected-(SW2-PadMP2)
- SW2 pad MP3: (no net) -> unconnected-(SW2-PadMP3)
- SW2 pad MP4: (no net) -> unconnected-(SW2-PadMP4)
- SW2 pad MP5: (no net) -> unconnected-(SW2-PadMP5)
- SW2 pad MP6: (no net) -> unconnected-(SW2-PadMP6)
- SW3 pad A: /Encoders/Encoder3/A1 -> /encoder2/A1
- SW3 pad B: /Encoders/Encoder3/B1 -> /encoder2/B1
- SW3 pad MP1: (no net) -> unconnected-(SW3-PadMP1)
- SW3 pad MP2: (no net) -> unconnected-(SW3-PadMP2)
- SW3 pad MP3: (no net) -> unconnected-(SW3-PadMP3)
- SW3 pad MP4: (no net) -> unconnected-(SW3-PadMP4)
- SW3 pad MP5: (no net) -> unconnected-(SW3-PadMP5)
- SW3 pad MP6: (no net) -> unconnected-(SW3-PadMP6)
- SW4 pad A: /Encoders/Encoder5/A1 -> /encoder3/A1
- SW4 pad B: /Encoders/Encoder5/B1 -> /encoder3/B1
- SW4 pad MP1: (no net) -> unconnected-(SW4-PadMP1)
- SW4 pad MP2: (no net) -> unconnected-(SW4-PadMP2)
- SW4 pad MP3: (no net) -> unconnected-(SW4-PadMP3)
- SW4 pad MP4: (no net) -> unconnected-(SW4-PadMP4)
- SW4 pad MP5: (no net) -> unconnected-(SW4-PadMP5)
- SW4 pad MP6: (no net) -> unconnected-(SW4-PadMP6)
- SW5 pad A: /Encoders/Encoder6/A1 -> /encoder4/A1
- SW5 pad B: /Encoders/Encoder6/B1 -> /encoder4/B1
- SW5 pad MP1: (no net) -> unconnected-(SW5-PadMP1)
- SW5 pad MP2: (no net) -> unconnected-(SW5-PadMP2)
- SW5 pad MP3: (no net) -> unconnected-(SW5-PadMP3)
- SW5 pad MP4: (no net) -> unconnected-(SW5-PadMP4)
- SW5 pad MP5: (no net) -> unconnected-(SW5-PadMP5)
- SW5 pad MP6: (no net) -> unconnected-(SW5-PadMP6)
- SW6 pad A: /Encoders/Encoder4/A1 -> /encoder7/A1
- SW6 pad B: /Encoders/Encoder4/B1 -> /encoder7/B1
- SW6 pad MP1: (no net) -> unconnected-(SW6-PadMP1)
- SW6 pad MP2: (no net) -> unconnected-(SW6-PadMP2)
- SW6 pad MP3: (no net) -> unconnected-(SW6-PadMP3)
- SW6 pad MP4: (no net) -> unconnected-(SW6-PadMP4)
- SW6 pad MP5: (no net) -> unconnected-(SW6-PadMP5)
- SW6 pad MP6: (no net) -> unconnected-(SW6-PadMP6)
- SW7 pad A: /Encoders/Encoder7/A1 -> /encoder5/A1
- SW7 pad B: /Encoders/Encoder7/B1 -> /encoder5/B1
- SW7 pad MP1: (no net) -> unconnected-(SW7-PadMP1)
- SW7 pad MP2: (no net) -> unconnected-(SW7-PadMP2)
- SW7 pad MP3: (no net) -> unconnected-(SW7-PadMP3)
- SW7 pad MP4: (no net) -> unconnected-(SW7-PadMP4)
- SW7 pad MP5: (no net) -> unconnected-(SW7-PadMP5)
- SW7 pad MP6: (no net) -> unconnected-(SW7-PadMP6)
- SW8 pad MP1: (no net) -> unconnected-(SW8-PadMP1)
- SW8 pad MP2: (no net) -> unconnected-(SW8-PadMP2)
- SW8 pad MP3: (no net) -> unconnected-(SW8-PadMP3)
- SW8 pad MP4: (no net) -> unconnected-(SW8-PadMP4)
- SW8 pad MP5: (no net) -> unconnected-(SW8-PadMP5)
- SW8 pad MP6: (no net) -> unconnected-(SW8-PadMP6)
- U3 pad 86: /Encoders/Encoder0/enc.s -> unconnected-(U3-LVDS_TX1_N-Pad86)
- U3 pad 87: /Encoders/Encoder0/enc.b -> unconnected-(U3-LVDS_TX1_P-Pad87)
- U3 pad 88: /Encoders/Encoder0/enc.a -> unconnected-(U3-LVDS_TX2_N-Pad88)
Routing:
- net /Encoders/Encoder0/enc.s: track 1.91 -> 0.00 mm
Other:
- board size 330.4 x 275 mm -> 173.4 x 182.9 mm

Commit message: Moved encoders around
Parts:
- removed SW1, SW2, SW3, SW5, SW6, SW7, SW8: RotaryEncoder_Switch, d-lev:PEC11S-929K
- added SW4: RotaryEncoder_Switch, d-lev:PEC11S-929K, F.Cu at (56.7, -19.1)
- added SW4: RotaryEncoder_Switch, d-lev:PEC11S-929K, F.Cu at (19.1, 40.2)
- added SW4: RotaryEncoder_Switch, d-lev:PEC11S-929K, F.Cu at (57.1, 18.0)
- added SW4: RotaryEncoder_Switch, d-lev:PEC11S-929K, F.Cu at (-57.6, -18.0)
- added SW4: RotaryEncoder_Switch, d-lev:PEC11S-929K, F.Cu at (-18.0, 40.6)
- added SW4: RotaryEncoder_Switch, d-lev:PEC11S-929K, F.Cu at (18.0, -41.1)
- added SW4: RotaryEncoder_Switch, d-lev:PEC11S-929K, F.Cu at (-57.1, 19.1)
- moved SW4 245.0 mm to (-19.1, -40.6), turned to 90 degrees
- moved DS2 51.5 mm to (0.00, 0.00)
- moved U3 11.9 mm to (140.8, 49.7)
Other:
- board size 173.4 x 182.9 mm -> 365.1 x 393.1 mm
