File: d-lev-main/dlev-mini.kicad_pcb (KiCad board)
At the start: 4 copper layers, 365.1 x 393.1 mm, 78 parts, among them J1 Conn_01x12_MountingPin, J2 Tag-Connect TC2030-NL, J3 S8B-PH-SM4-TB, J4 S8B-PH-SM4-TB, J5 Conn_01x06_MountingPin, Q2 MMBT3904, Q3 BSS138, Q4 BSS138, Q5 BSS138, SW4 RotaryEncoder_Switch, U1 25LCxxx, U2 AMS1117-3.3, U3 AC608

Commit message: start routing
* add simple knob model
* place encoders
* change display to use SMT female headers and SMTSO screw holes
* rotate fpga model 90 degrees
Parts:
- removed the SW4 at (56.7, -19.1)
- removed the SW4 at (19.1, 40.2)
- removed the SW4 at (57.1, 18.0)
- removed the SW4 at (-57.6, -18.0)
- removed the SW4 at (-18.0, 40.6)
- removed the SW4 at (18.0, -41.1)
- removed the SW4 at (-57.1, 19.1)
- removed the SW4 at (-19.1, -40.6)
- added H5: M3 Standoff, d-lev:SMTSO-M3, F.Cu at (46.5, -97.5)
- added H6: M3 Standoff, d-lev:SMTSO-M3, F.Cu at (-46.5, -97.5)
- added H7: M3 Standoff, d-lev:SMTSO-M3, F.Cu at (-46.5, -42.5)
- added H8: M3 Standoff, d-lev:SMTSO-M3, F.Cu at (46.5, -42.5)
- added RN10: 4.7k, Resistor_SMD:R_Array_Concave_4x0603, F.Cu at (6.15, 2.00)
- added RN9: 4.7k, Resistor_SMD:R_Array_Concave_4x0603, F.Cu at (2.00, 2.00)
- added SW1: RotaryEncoder_Switch, d-lev:PEC11S-929K, F.Cu at (-70.6, -32.2)
- added SW2: RotaryEncoder_Switch, d-lev:PEC11S-929K, F.Cu at (-35.6, -14.7)
- added SW3: RotaryEncoder_Switch, d-lev:PEC11S-929K, F.Cu at (-70.6, 2.82)
- added SW4: RotaryEncoder_Switch, d-lev:PEC11S-929K, F.Cu at (-35.6, 20.3)
- added SW5: RotaryEncoder_Switch, d-lev:PEC11S-929K, F.Cu at (70.6, -32.2)
- added SW6: RotaryEncoder_Switch, d-lev:PEC11S-929K, F.Cu at (35.6, -14.7)
- added SW7: RotaryEncoder_Switch, d-lev:PEC11S-929K, F.Cu at (70.6, 2.82)
- added SW8: RotaryEncoder_Switch, d-lev:PEC11S-929K, F.Cu at (35.6, 20.3)
- C1, C11, C12, C13, C14, C15, C16, C17, C18, C19, C2, C20, C21, C3, C4, C5, C6, C9: footprint Capacitor_SMD:C_0805_2012Metric_Pad1.18x1.45mm_HandSolder -> Capacitor_SMD:C_0603_1608Metric
- DS2: footprint d-lev:ERM2004-0 -> d-lev:ERM2004-2
- RN1, RN2, RN3, RN4, RN5, RN6, RN7, RN8: value 10k -> 4.7k
- U3: footprint d-lev:ac608 -> d-lev:ac608-toponly
- moved J4 246.8 mm to (-60.0, -83.8), turned to -90 degrees
- moved C2 246.8 mm to (-65.0, -44.0), turned to 135 degrees
- moved RN1 244.2 mm to (-61.0, -41.0), turned to 45 degrees
- moved C1 234.9 mm to (-58.0, -37.0), turned to -45 degrees
- moved J5 207.3 mm to (22.9, -86.4), turned to 180 degrees
- moved J3 206.9 mm to (60.0, -83.8), turned to 90 degrees
- moved U3 158.2 mm to (0.00, -22.4), turned to 45 degrees
- moved C3 155.2 mm to (17.8, 81.6)
- moved C4 155.2 mm to (17.8, 84.6)
- moved RN2 151.0 mm to (22.3, 82.5)
- moved C5 148.1 mm to (28.7, 81.6)
- moved C6 148.1 mm to (28.7, 84.6)
- moved RN3 145.0 mm to (33.2, 82.5)
- moved C20 138.5 mm to (17.8, 89.6)
- moved C21 138.5 mm to (17.8, 92.6)
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Connections:
- U3 pad 1: unconnected-(U3-IO_T14-Pad1) -> (no net)
- U3 pad 10: unconnected-(U3-IO_L15-Pad10) -> (no net)
- U3 pad 100: unconnected-(U3-IO_R3-Pad100) -> (no net)
- U3 pad 101: unconnected-(U3-IO_T3-Pad101) -> (no net)
- U3 pad 102: unconnected-(U3-IO_R4-Pad102) -> (no net)
- U3 pad 103: unconnected-(U3-IO_T4-Pad103) -> (no net)
- U3 pad 104: unconnected-(U3-IO_R5-Pad104) -> (no net)
- U3 pad 105: unconnected-(U3-IO_T5-Pad105) -> (no net)
- U3 pad 106: +3V3 -> (no net)
- U3 pad 107: GND -> (no net)
- U3 pad 108: unconnected-(U3-IO_R6-Pad108) -> (no net)
- U3 pad 109: unconnected-(U3-IO_T6-Pad109) -> (no net)
- U3 pad 11: unconnected-(U3-IO_L16-Pad11) -> (no net)
- U3 pad 110: unconnected-(U3-IO_R7-Pad110) -> (no net)
- U3 pad 111: unconnected-(U3-IO_T7-Pad111) -> (no net)
- U3 pad 112: unconnected-(U3-I_R8-Pad112) -> (no net)
- U3 pad 113: unconnected-(U3-I_T8-Pad113) -> (no net)
- U3 pad 114: unconnected-(U3-I_R9-Pad114) -> (no net)
- U3 pad 115: unconnected-(U3-I_T9-Pad115) -> (no net)
- U3 pad 116: unconnected-(U3-IO_R10-Pad116) -> (no net)
- U3 pad 117: unconnected-(U3-IO_T10-Pad117) -> (no net)
- U3 pad 118: unconnected-(U3-IO_R11-Pad118) -> (no net)
- U3 pad 119: unconnected-(U3-IO_T11-Pad119) -> (no net)
- U3 pad 12: unconnected-(U3-IO_P11-Pad12) -> (no net)
- U3 pad 120: unconnected-(U3-IO_R12-Pad120) -> (no net)
- U3 pad 121: unconnected-(U3-IO_T12-Pad121) -> (no net)
- U3 pad 122: unconnected-(U3-IO_R13-Pad122) -> (no net)
- U3 pad 123: unconnected-(U3-IO_T13-Pad123) -> (no net)
- U3 pad 124: unconnected-(U3-IO_R14-Pad124) -> (no net)
- U3 pad 13: unconnected-(U3-IO_N11-Pad13) -> (no net)
- U3 pad 14: +3V3 -> (no net)
- U3 pad 15: GND -> (no net)
- U3 pad 16: unconnected-(U3-IO_N12-Pad16) -> (no net)
- U3 pad 17: unconnected-(U3-IO_P14-Pad17) -> (no net)
- U3 pad 18: unconnected-(U3-IO_N14-Pad18) -> (no net)
- U3 pad 19: unconnected-(U3-IO_L13-Pad19) -> (no net)
- U3 pad 2: unconnected-(U3-IO_T15-Pad2) -> (no net)
- U3 pad 20: unconnected-(U3-IO_K16-Pad20) -> (no net)
- U3 pad 21: unconnected-(U3-IO_J15-Pad21) -> (no net)
- U3 pad 22: unconnected-(U3-IO_J16-Pad22) -> (no net)
- U3 pad 23: unconnected-(U3-IO_L14-Pad23) -> (no net)
- U3 pad 24: unconnected-(U3-IO_J14-Pad24) -> (no net)
- U3 pad 25: unconnected-(U3-IO_K15-Pad25) -> (no net)
- U3 pad 26: unconnected-(U3-IO_F16-Pad26) -> (no net)
- U3 pad 27: unconnected-(U3-IO_G15-Pad27) -> (no net)
- U3 pad 28: unconnected-(U3-IO_F15-Pad28) -> (no net)
- U3 pad 29: unconnected-(U3-I_E16-Pad29) -> (no net)
- U3 pad 3: unconnected-(U3-IO_R16-Pad3) -> (no net)
- U3 pad 30: unconnected-(U3-IO_D16-Pad30) -> (no net)
- U3 pad 31: unconnected-(U3-IO_D15-Pad31) -> (no net)
- U3 pad 32: unconnected-(U3-IO_C16-Pad32) -> (no net)
- U3 pad 33: unconnected-(U3-IO_C15-Pad33) -> (no net)
- U3 pad 34: unconnected-(U3-IO_B16-Pad34) -> (no net)
- U3 pad 35: unconnected-(U3-IO_J13-Pad35) -> (no net)
- U3 pad 36: unconnected-(U3-IO_G16-Pad36) -> (no net)
- U3 pad 37: unconnected-(U3-IO_F8-Pad37) -> (no net)
- U3 pad 38: unconnected-(U3-IO_F13-Pad38) -> (no net)
- U3 pad 39: unconnected-(U3-IO_F14-Pad39) -> (no net)
- U3 pad 4: unconnected-(U3-IO_P15-Pad4) -> (no net)
- U3 pad 40: unconnected-(U3-IO_F9-Pad40) -> (no net)
- U3 pad 41: unconnected-(U3-IO_E11-Pad41) -> (no net)
- U3 pad 42: unconnected-(U3-I_A9-Pad42) -> (no net)
- U3 pad 43: unconnected-(U3-I_B9-Pad43) -> (no net)
- U3 pad 44: unconnected-(U3-IO_C9-Pad44) -> (no net)
- U3 pad 45: unconnected-(U3-I_A8-Pad45) -> (no net)
- U3 pad 46: unconnected-(U3-IO_D9-Pad46) -> (no net)
- U3 pad 47: unconnected-(U3-I_B8-Pad47) -> (no net)
- U3 pad 48: +3V3 -> (no net)
- U3 pad 49: GND -> (no net)
- U3 pad 5: unconnected-(U3-IO_P16-Pad5) -> (no net)
- U3 pad 50: unconnected-(U3-I_E1-Pad50) -> (no net)
- U3 pad 51: unconnected-(U3-IO_B1-Pad51) -> (no net)
- U3 pad 52: unconnected-(U3-IO_C2-Pad52) -> (no net)
- U3 pad 53: unconnected-(U3-IO_D1-Pad53) -> (no net)
- U3 pad 54: unconnected-(U3-IO_F3-Pad54) -> (no net)
- U3 pad 55: unconnected-(U3-IO_F2-Pad55) -> (no net)
- U3 pad 56: unconnected-(U3-IO_F1-Pad56) -> (no net)
- U3 pad 57: unconnected-(U3-IO_G5-Pad57) -> (no net)
- U3 pad 58: unconnected-(U3-IO_G2-Pad58) -> (no net)
- U3 pad 59: unconnected-(U3-IO_G1-Pad59) -> (no net)
- U3 pad 6: unconnected-(U3-IO_N15-Pad6) -> (no net)
- U3 pad 60: /FPGA/TCK -> (no net)
- U3 pad 61: /FPGA/TDI -> (no net)
- U3 pad 62: /FPGA/TMS -> (no net)
- U3 pad 63: +2V5 -> (no net)
- U3 pad 64: /FPGA/TDO -> (no net)
- U3 pad 65: unconnected-(U3-IO_K5-Pad65) -> (no net)
- U3 pad 66: unconnected-(U3-IO_L4-Pad66) -> (no net)
- U3 pad 67: unconnected-(U3-IO_M6-Pad67) -> (no net)
- U3 pad 68: unconnected-(U3-IO_N3-Pad68) -> (no net)
- U3 pad 69: unconnected-(U3-IO_N5-Pad69) -> (no net)
- U3 pad 7: unconnected-(U3-IO_N16-Pad7) -> (no net)
- U3 pad 70: unconnected-(U3-IO_P3-Pad70) -> (no net)
- U3 pad 71: unconnected-(U3-IO_L7-Pad71) -> (no net)
- U3 pad 72: unconnected-(U3-IO_N6-Pad72) -> (no net)
- U3 pad 73: GND -> (no net)
- U3 pad 74: +1V2 -> (no net)
- U3 pad 75: unconnected-(U3-IO_P6-Pad75) -> (no net)
- U3 pad 76: unconnected-(U3-IO_M7-Pad76) -> (no net)
- U3 pad 77: unconnected-(U3-IO_M8-Pad77) -> (no net)
- U3 pad 78: +3V3 -> (no net)
- U3 pad 79: GND -> (no net)
- U3 pad 8: unconnected-(U3-I_M15-Pad8) -> (no net)
- U3 pad 80: unconnected-(U3-IO_P8-Pad80) -> (no net)
- U3 pad 81: unconnected-(U3-IO_N8-Pad81) -> (no net)
- U3 pad 82: unconnected-(U3-IO_L8-Pad82) -> (no net)
- U3 pad 83: unconnected-(U3-IO_N9-Pad83) -> (no net)
- U3 pad 84: unconnected-(U3-IO_P9-Pad84) -> (no net)
- U3 pad 85: unconnected-(U3-IO_M10-Pad85) -> (no net)
- U3 pad 86: unconnected-(U3-LVDS_TX1_N-Pad86) -> (no net)
- U3 pad 87: unconnected-(U3-LVDS_TX1_P-Pad87) -> (no net)
- U3 pad 88: unconnected-(U3-LVDS_TX2_N-Pad88) -> (no net)
- U3 pad 89: unconnected-(U3-LVDS_TX2_P-Pad89) -> (no net)
- U3 pad 9: unconnected-(U3-I_M16-Pad9) -> (no net)
- U3 pad 90: unconnected-(U3-LVDS_TX3_N-Pad90) -> (no net)
- U3 pad 91: unconnected-(U3-LVDS_TX3_P-Pad91) -> (no net)
- U3 pad 92: unconnected-(U3-LVDS_RXCLK_N-Pad92) -> (no net)
- U3 pad 93: unconnected-(U3-LVDS_RXCLK_P-Pad93) -> (no net)
- U3 pad 94: unconnected-(U3-LVDS_TX4_N-Pad94) -> (no net)
- U3 pad 95: unconnected-(U3-LVDS_TX4_P-Pad95) -> (no net)
- U3 pad 96: unconnected-(U3-LVDS_TX5_N-Pad96) -> (no net)
- U3 pad 97: unconnected-(U3-LVDS_TX5_P-Pad97) -> (no net)
- U3 pad 98: unconnected-(U3-IO_R1-Pad98) -> (no net)
- U3 pad 99: unconnected-(U3-IO_T2-Pad99) -> (no net)
Routing:
- net /encoder1/A1: track 0.00 -> 6.45 mm
- net /encoder1/B1: track 0.00 -> 5.75 mm
- net enc_2.a: track 0.00 -> 5.74 mm
- net enc_2.b: track 0.00 -> 3.36 mm
Other:
- board size 365.1 x 393.1 mm -> 171.4 x 146.7 mm
