File: d-lev-main/d-lev-main.kicad_sch (KiCad schematic)
At the start: 49 parts, among them J1 S6B-PH-SM4-TB, J2 S8B-PH-SM4-TB, J3 S8B-PH-SM4-TB, J4 S12B-PH-SM4-TB, U3 AMS1117-3.3

Commit message: Add iBOMs and additional part numbers
Parts:
- C11, C9: MPN (none) -> GRM188R71E104KA01D; Notes (none) -> Common; Supplier (none) -> Digi-Key; Supplier URL (none) -> https://www.digikey.com/en/products/detail/murata-electroni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
- C19, C20: Supplier (none) -> Mouser; Supplier URL (none) -> https://www.mouser.com/ProductDetail/Samsung-Electro-Mechan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
- CRIMPED_LEAD1, CRIMPED_LEAD2, CRIMPED_LEAD4: DNP (none) -> Y
- H1, H2, H7, H8: Supplier (none) -> Aliexpress; Supplier URL (none) -> https://www.aliexpress.us/item/3256803593893401.html
- J1: MPN (none) -> S6B-PH-SM4-TB; Supplier (none) -> Digi-Key; Supplier Alt (none) -> Aliexpress; Supplier Alt URL (none) -> https://www.aliexpress.us/item/3256805219782364.html; Supplier URL (none) -> https://www.digikey.com/en/products/detail/jst-sales-americ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
- J2, J3: MPN (none) -> S8B-PH-SM4-TB; Supplier (none) -> Digi-Key; Supplier Alt (none) -> Aliexpress; Supplier Alt URL (none) -> https://www.aliexpress.us/item/3256805227213161.html; Supplier URL (none) -> https://www.digikey.com/en/products/detail/jst-sales-americ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
- J4: MPN (none) -> S12B-PH-SM4-TB; Supplier (none) -> Digi-Key; Supplier Alt (none) -> Aliexpress; Supplier Alt URL (none) -> https://www.aliexpress.us/item/3256805244385531.html; Supplier URL (none) -> https://www.digikey.com/en/products/detail/jst-sales-americ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
- R10, R12: MPN (none) -> RC0603FR-13110RL; Supplier (none) -> Digi-Key; Supplier URL (none) -> https://www.digikey.com/en/products/detail/yageo/RC0603FR-1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; Tolerance (none) -> 1%
- R11, R9: MPN (none) -> RC0603FR-07221RL; Supplier (none) -> Digi-Key; Supplier URL (none) -> https://www.digikey.com/en/products/detail/yageo/RC0603FR-0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; Tolerance (none) -> 1%
- TP10, TP11, TP12, TP13, TP14, TP15, TP16, TP17, TP18, TP19, TP20, TP21, TP22, TP23, TP24, TP25, TP26, TP27: DNP (none) -> Y; now left out of the parts list
- TP3: value GND -> TestPoint; DNP (none) -> Y
- TP3: value VDD -> TestPoint; DNP (none) -> Y; now left out of the parts list
- U3: Supplier (none) -> Mouser
- WIRE_HOUSING1, WIRE_HOUSING2: DNP (none) -> Y; Notes (none) -> PH2.0; Supplier (none) -> Aliexpress; Supplier URL (none) -> https://www.aliexpress.us/item/3256804371551423.html
- WIRE_HOUSING4: DNP (none) -> Y; Notes (none) -> PH2.0, different directions; Supplier (none) -> Aliexpress; Supplier URL (none) -> https://www.aliexpress.us/item/3256804371551423.html
Other:
- note added: "NOTE: GET THE REVERSE WIRED VERSION TO CONNECT WITH TUNER REV1"
