File: d-lev_afe-antenna/d-lev_afe-antenna.kicad_pcb (KiCad board)
At the start: 2 copper layers, 282 x 177.5 mm, 25 parts, among them J1 S7B-PH-SM4-TB, Q1 MMBT3904, Q2 MMBT3906, U1 74AHC04, U2 HT7533-1-SOT89, U3 SRV05-4

Commit message: Many changes
Reorganized libraries to share between projects
Set up JLC 2- and 4- layer design rules
Finished copying over most of the schematic (excluding I/O board)
Parts:
- added H3: Standoff_2, theremin:SMTSO-M4, B.Cu at (168.8, 45.6)
- H1, H2: moved to B.Cu
- J1: value S7B-PH-SM4-TB -> Conn_01x08; footprint Connector_JST:JST_PH_S7B-PH-SM4-TB_1x07-1MP_P2.00mm_Horizontal -> Connector_JST:JST_PH_S8B-PH-SM4-TB_1x08-1MP_P2.00mm_Horizontal
- moved H1 138.1 mm to (188.1, 80.2), turned to 180 degrees
- moved H2 121.9 mm to (168.8, 106.2), turned to 180 degrees
- moved L1 121.9 mm to (168.8, 80.7)
- moved C8 111.1 mm to (156.4, 88.7), turned to 135 degrees
- moved C4 110.1 mm to (159.4, 71.2), turned to -135 degrees
- moved Q2 109.5 mm to (155.9, 70.9), turned to 45 degrees
- moved C7 109.5 mm to (153.7, 86.1), turned to 135 degrees
- moved Q1 109.3 mm to (158.8, 68.0), turned to 45 degrees
- moved R2 109.0 mm to (152.7, 74.4), turned to -45 degrees
- moved R3 108.8 mm to (154.0, 73.1), turned to 135 degrees
- moved C6 108.4 mm to (154.7, 89.9), turned to 135 degrees
- moved R1 108.0 mm to (138.2, 79.2)
- moved J1 107.2 mm to (130.7, 80.2)
- moved C1 106.9 mm to (138.7, 91.2)
- moved C2 106.9 mm to (142.7, 87.2)
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Connections:
- H1 pad 1: unconnected-(H1-Pad1) -> L_OUT
- J1 pad 1: ZERO -> GND
- J1 pad 2: GND -> ZERO
- J1 pad 3: QUAD -> GND
- J1 pad 4: GND -> SQ
- J1 pad 5: SQ -> GND
- J1 pad 6: GND -> QUAD
- J1 pad 7: +5V -> GND
- U1 pad 1: GND -> Net-(R5-Pad2)
- U1 pad 10: Net-(R7-Pad1) -> Net-(R2-Pad1)
- U1 pad 11: Net-(R6-Pad1) -> Net-(R1-Pad2)
- U1 pad 12: Net-(R2-Pad1) -> Net-(R7-Pad1)
- U1 pad 13: Net-(R1-Pad2) -> Net-(R6-Pad1)
- U1 pad 2: unconnected-(U1-Pad2) -> Net-(R6-Pad1)
- U1 pad 3: Net-(R5-Pad2) -> GND
- U1 pad 4: Net-(R6-Pad1) -> unconnected-(U1-Pad4)
Routing:
- net +3V3: track 57.6 -> 24.3 mm, vias 3 -> 4
- net GND: track 36.3 -> 8.54 mm, vias 3 -> 0
- net L_OUT: track 27.2 -> 51.2 mm, vias 2 -> 0
- net L_IN: track 7.01 -> 17.9 mm
- net Net-(R3-Pad2): track 5.21 -> 9.78 mm
- net Net-(R5-Pad2): track 5.33 -> 6.85 mm
- net Net-(R2-Pad1): track 11.5 -> 12.5 mm
- net /C_DIV: track 18.7 -> 19.4 mm, vias 0 -> 2
- net Net-(R7-Pad1): track 3.98 -> 4.58 mm
- net Net-(R1-Pad2): track 4.05 -> 3.45 mm
- added copper zone on B.Cu, net +3V3
- removed copper zone on B.Cu, net L_IN
Other:
- board size 282 x 177.5 mm -> 109.4 x 93 mm
- rule pad_to_mask_clearance: 0 -> 0.05
- board text added: "L_OUT Drive side - near antenna mount"
- board text added: "Sense side Minimize copper"
