File: d-lev-io/midi.kicad_sch (KiCad schematic)
At the start: 9 parts, among them J3 AudioJack3, J3 MIDI_IN_JACK, J4 DIN-41524, U2 6N137

Commit message: more minor pusharounds and updates
Parts:
- J3: footprint (none) -> Connector_Audio:Jack_3.5mm_CUI_SJ-3523-SMT_Horizontal
- J3: value MIDI_IN_JACK -> MIDI_OUT_JACK; footprint (none) -> Connector_Audio:Jack_3.5mm_CUI_SJ-3523-SMT_Horizontal
- R3, R4, R5: footprint (none) -> Resistor_SMD:R_0603_1608Metric
Changed lines of the file:
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@@
       (effects (font (size 1.27 1.27)) (justify right))
     )
-    (property "Footprint" "" (at 131.953 111.125 90)
+    (property "Footprint" "Resistor_SMD:R_0603_1608Metric" (at 131.953 111.125 90)
       (effects (font (size 1.27 1.27)) hide)
     )
@@
       (effects (font (size 1.27 1.27)) (justify right))
     )
-    (property "Footprint" "" (at 145.923 116.84 90)
+    (property "Footprint" "Resistor_SMD:R_0603_1608Metric" (at 145.923 116.84 90)
       (effects (font (size 1.27 1.27)) hide)
     )
@@
       (effects (font (size 1.27 1.27)))
     )
-    (property "Footprint" "" (at 97.155 129.413 90)
+    (property "Footprint" "Resistor_SMD:R_0603_1608Metric" (at 97.155 129.413 90)
       (effects (font (size 1.27 1.27)) hide)
     )
@@
       (effects (font (size 1.27 1.27)))
     )
-    (property "Footprint" "" (at 169.545 126.365 0)
+    (property "Footprint" "Connector_Audio:Jack_3.5mm_CUI_SJ-3523-SMT_Horizontal" (at 169.545 126.365 0)
       (effects (font (size 1.27 1.27)) hide)
     )
@@
       (effects (font (size 1.27 1.27)))
     )
-    (property "Value" "MIDI_IN_JACK" (at 81.28 68.58 0)
-      (effects (font (size 1.27 1.27)))
-    )
-    (property "Footprint" "" (at 83.185 74.295 0)
-      (effects (font (size 1.27 1.27)) hide)
-    )
+    (property "Value" "MIDI_OUT_JACK" (at 81.28 68.58 0)
+      (effects (font (size 1.27 1.27)))
+    )
+    (property "Footprint" "Connector_Audio:Jack_3.5mm_CUI_SJ-3523-SMT_Horizontal" (at 83.185 74.295 0)
+      (effects (font (size 1.27 1.27)) hide)
+    )
