File: d-lev-io/d-lev-io.kicad_pcb (KiCad board)
At the start: 2 copper layers, 175.3 x 110.6 mm, 131 parts, among them IC1 ES9010K2M, IC3 MAX97220AETE+T, J1 USB_C_Receptacle_USB2.0, J2 PJ-059A, J3 Conn_01x12_MountingPin, J4 MIDI_OUT_JACK, J5 PROG_HDR, J6 HEADPHONE, SW1 SW_Push, SW2 SW_Push, SW3 SW_Push, U1 ATSAMD11D14A-M, U2 TPS54202DDC, U3 ADP151-3.3, U5 AP2112K-3.3, U6 74AHC1G126, X1 7M-50.000MAAJ-T

Commit message: many board updates
Parts:
- removed D5: STATUS_2, LED_SMD:LED_0603_1608Metric
- removed JP2: BUCK_VERSION, Jumper:SolderJumper-2_P1.3mm_Bridged_RoundedPad1.0x1.5mm
- removed JP3: JUMP_VBUCK, Jumper:SolderJumper-2_P1.3mm_Bridged_RoundedPad1.0x1.5mm
- removed JP4: JUMP_VBUS, Jumper:SolderJumper-2_P1.3mm_Bridged_RoundedPad1.0x1.5mm
- removed JP7: ADDRSEL, Jumper:SolderJumper-2_P1.3mm_Bridged_RoundedPad1.0x1.5mm
- removed R11: 510k, Resistor_SMD:R_0805_2012Metric
- removed R12: 105k, Resistor_SMD:R_0805_2012Metric
- removed R42, R44: 0, Resistor_SMD:R_0603_1608Metric
- removed RV2: 20K, theremin:RK10J12R0A0B
- removed the U3 at (104.5, 140.2)
- added C33: 4.7n, Capacitor_SMD:C_0603_1608Metric, F.Cu at (87.3, 93.0)
- added C34: 100n, Capacitor_SMD:C_0603_1608Metric, F.Cu at (94.7, 94.1)
- added C37: 4.7n, Capacitor_SMD:C_0603_1608Metric, F.Cu at (87.3, 95.2)
- added C40: 100n, Capacitor_SMD:C_0603_1608Metric, F.Cu at (141.9, 67.0)
- added C41: 10u, Capacitor_SMD:C_0603_1608Metric, F.Cu at (197.8, 64.8)
- added C42: .1u, Capacitor_SMD:C_0603_1608Metric, F.Cu at (197.7, 66.7)
- added C43: 1u, Capacitor_SMD:C_0603_1608Metric, F.Cu at (152.1, 81.2)
- added H1: MountingHole_Pad, theremin:SMTSO-M3, F.Cu at (236.9, 96.2)
- added H2: MountingHole_Pad, theremin:SMTSO-M3, F.Cu at (236.9, 57.0)
- added H3: MountingHole_Pad, theremin:MicStandHole, F.Cu at (101.4, 76.7)
- added H4: MountingHole_Pad, theremin:SMTSO-M3, F.Cu at (74.8, 57.0)
- added H5: MountingHole_Pad, theremin:SMTSO-M3, F.Cu at (74.8, 96.2)
- added R17: 27, Resistor_SMD:R_0603_1608Metric, F.Cu at (137.5, 89.2)
- added R36: 27, Resistor_SMD:R_0603_1608Metric, F.Cu at (137.4, 96.0)
- added R37: 75, Resistor_SMD:R_0603_1608Metric, F.Cu at (84.9, 95.5)
- added R38: 100k, Resistor_SMD:R_0603_1608Metric, F.Cu at (91.1, 91.4)
- added R39: 220, Resistor_SMD:R_0603_1608Metric, F.Cu at (88.0, 91.4)
- added R40: 220, Resistor_SMD:R_0603_1608Metric, F.Cu at (88.0, 96.8)
- added R41: 100k, Resistor_SMD:R_0603_1608Metric, F.Cu at (91.1, 96.8)
- added R43: 0, Resistor_SMD:R_0603_1608Metric, F.Cu at (157.6, 77.7)
- added TP25: VBUCK, TestPoint:TestPoint_Pad_D1.5mm, B.Cu at (317.7, 45.5)
- added U4: 74LVC2GU04, Package_TO_SOT_SMD:SOT-23-6, F.Cu at (91.1, 94.1)
- added VR1: RK09711110EL, theremin:RK09711110EL, F.Cu at (178.4, 97.1)
- C24: value .1u -> 1u
- IC3: value MAX97220AETE+T -> MAX97220C/MAX97220D
- J5: moved to B.Cu
- R18: value 10 -> 220
- R28: value 1k -> 75
- R8: value 33 -> 220
- TP2, TP23, TP3, TP4, TP5: moved to F.Cu
- moved TP1 262.6 mm to (326.2, 49.6), turned to -90 degrees
- moved TP2 179.6 mm to (250.6, 91.1)
- moved J2 178.9 mm to (228.0, 86.3), turned to 90 degrees
- moved R15 164.6 mm to (227.2, 68.1), turned to 135 degrees
- moved R14 163.1 mm to (225.7, 69.5), turned to -45 degrees
- moved C13 162.2 mm to (229.4, 75.8), turned to 90 degrees
- moved R13 160.5 mm to (223.2, 68.1), turned to 45 degrees
- moved C14 154.0 mm to (226.7, 76.2), turned to 90 degrees
- moved C17 148.9 mm to (216.5, 72.9)
- moved C18 148.8 mm to (216.4, 76.2)
- moved C15 148.1 mm to (220.9, 76.1), turned to -90 degrees
- moved C16 147.7 mm to (224.6, 71.0), turned to -45 degrees
- moved R4 147.0 mm to (231.8, 66.4), turned to 0 degrees
- moved U2 146.2 mm to (223.7, 75.8), turned to 90 degrees
- moved R1 146.2 mm to (239.0, 75.1), turned to 180 degrees
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Connections:
- net /DAC/OUT_SE.G renamed /DAC/AMP_SGND
- net /SAMD11/USB.DM renamed /SAMD11/USB.DN
- net Net-(J1-D+-PadA6) renamed /UINP
- net Net-(J1-D--PadA7) renamed /UINN
- C10 pad 1: Net-(C10-Pad1) -> /DAC/DAC.XI
- C2 pad 2: +5V -> SWITCH_LOW
- C23 pad 2: +5V -> VDD
- C26 pad 2: +5V -> VDD
- C28 pad 2: Net-(RN1-R4.1) -> /DAC/IN_BAL.L+
- C29 pad 2: Net-(RN1-R1.1) -> /DAC/IN_BAL.R+
- C3 pad 2: +5V -> SWITCH_LOW
- C30 pad 2: Net-(RN1-R3.1) -> /DAC/IN_BAL.L-
- C32 pad 2: Net-(RN1-R2.1) -> /DAC/IN_BAL.R-
- C36 pad 1: /DAC/AMP_PVDD -> +3.3VA
- C39 pad 1: /DAC/AMP_PVDD -> +3.3VA
- C4 pad 2: +5V -> SWITCH_LOW
- C5 pad 2: +5V -> SWITCH_LOW
- C6 pad 2: +5V -> SWITCH_LOW
- C7 pad 2: +5V -> SWITCH_LOW
- D2 pad 1: Net-(D2-K) -> Net-(D1-K)
- FB1 pad 1: Net-(JP3-B) -> Net-(D1-K)
- FB1 pad 2: +5V -> SWITCH_LOW
- IC1 pad 24: /DAC/DAC.GPIO -> /DAC/DAC_GPIO
- IC1 pad 28: /DAC/DAC.RESET -> /DAC/DAC_RESET
- IC3 pad 1: /DAC/AMP_PVDD -> +3.3VA
- IC3 pad 10: /DAC/OUT_SE.R -> /DAC/OUT_SE_R
- IC3 pad 12: /DAC/OUT_SE.L -> /DAC/OUT_SE_L
- IC3 pad 13: /DAC/AMP_PVDD -> +3.3VA
- IC3 pad 9: /DAC/AMP_PVDD -> +3.3VA
- J3 pad 12: +5V -> VDD
- R19 pad 2: /DAC/AMP_PVDD -> +3.3VA
- R28 pad 1: Net-(D5-A) -> spdif_line
- R28 pad 2: /SAMD11/STATUS_LED_2 -> GND
- R31 pad 2: Net-(C9-Pad1) -> /DAC/DAC.XO
- R8 pad 1: +3V3 -> VDD
- TP18 pad 1: /SAMD11/ESS_SHDN -> /DAC/DAC_RESET
- TP19 pad 1: /SAMD11/ESS_GPIO -> /DAC/DAC_GPIO
- TP20 pad 1: /SAMD11/HPA_SHDN -> /DAC/HPA_SHDN
- TP3 pad 1: +5V -> VDD
- TP6 pad 1: +5V -> VDD
- U1 pad 14: /SAMD11/STATUS_LED_2 -> /DAC/DAC_GPIO
- U1 pad 2: /SAMD11/HPA_SHDN -> /DAC/HPA_SHDN
- U1 pad 5: /SAMD11/ESS_SHDN -> /DAC/DAC_RESET
- U1 pad 6: /SAMD11/ESS_GPIO -> /SAMD11/VOLUME_POT
- U2 pad 5: Net-(JP2-B) -> unconnected-(U2-EN-Pad5)
- U5 pad 1: +5V -> VDD
- U5 pad 3: +5V -> VDD
- U6 pad 1: +3V3 -> VDD
- U6 pad 5: +3V3 -> VDD
- X1 pad 2: Net-(C10-Pad1) -> GND
- X1 pad 4: Net-(C9-Pad1) -> GND
Routing:
- net GND: track 0.00 -> 69.6 mm, vias 0 -> 126
- net Net-(D1-K): track 0.00 -> 39.8 mm
- net VBUS: track 0.00 -> 30.8 mm, vias 0 -> 2
- net /Buck/VOUT: track 0.00 -> 25.9 mm, vias 0 -> 2
- net Net-(U2-SW): track 0.00 -> 20.6 mm
- net /SAMD11/USB.DN: track 0.00 -> 20.0 mm, vias 0 -> 1
- net /SAMD11/USB.DP: track 0.00 -> 19.7 mm, vias 0 -> 1
- net +12V: track 0.00 -> 19.2 mm
- net Net-(J6-PadR): track 0.00 -> 17.3 mm
- net +3.3VA: track 0.00 -> 15.3 mm, vias 0 -> 8
- net SWITCH_LOW: track 0.00 -> 15.1 mm
- net Net-(J4-PadR): track 0.00 -> 12.0 mm
- net VDD: track 0.00 -> 11.5 mm, vias 0 -> 12
- net Net-(J1-CC2): track 0.00 -> 10.2 mm
- net /DAC/DAC.XI: track 0.00 -> 9.68 mm
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- added copper zone on F.Cu, net +3.3VA
- added copper zone on In2.Cu, net +3.3VA
- added copper zone on F.Cu, net +3V3
- added copper zone on In2.Cu, net +3V3
- added copper zone on B.Cu, net GND
- added copper zone on F.Cu, net GND
- added copper zone on In1.Cu, net GND
- added copper zone on In2.Cu, net GND
- added copper zone on F.Cu, net GNDA
- added copper zone on F.Cu, net SWITCH_LOW
- added copper zone on B.Cu, net VDD
- added copper zone on F.Cu, net VDD
Other:
- board size 175.3 x 110.6 mm -> 175.3 x 50.1 mm
- copper layers 2 -> 4
- rule solder_mask_min_width: 0.2 -> 0.15
- board text added: "TODO: decide on how to handle analog grounding"
- board text added: "TODO: review Schematic Checklist p.1112"

Commit message: more routing
Parts:
- removed NT1: NetTie_2, NetTie:NetTie-2_SMD_Pad0.5mm
- added R11: 511k, Resistor_SMD:R_0603_1608Metric, F.Cu at (215.7, 90.8)
- added R12: 105k, Resistor_SMD:R_0603_1608Metric, F.Cu at (215.7, 94.0)
- TP1, TP18, TP24, TP25: moved to F.Cu
- moved JP1 123.9 mm to (116.7, 95.3)
- moved JP5 123.9 mm to (116.7, 98.9), turned to 0 degrees
- moved R9 111.8 mm to (132.7, 98.4)
- moved R23 111.4 mm to (116.8, 83.7), turned to 180 degrees
- moved D4 111.4 mm to (117.1, 87.0), turned to 180 degrees
- moved R27 111.4 mm to (120.9, 99.0), turned to 180 degrees
- moved JP6 110.9 mm to (120.1, 85.3)
- moved TP1 109.4 mm to (221.2, 80.1)
- moved R26 107.3 mm to (120.9, 95.6), turned to -135 degrees
- moved R10 104.6 mm to (121.6, 91.2)
- moved SW3 101.3 mm to (117.4, 91.4)
- moved SW2 100.6 mm to (128.4, 99.0), turned to 0 degrees
- moved TP25 99.1 mm to (220.9, 66.8)
- moved R16 97.4 mm to (117.1, 85.4), turned to 0 degrees
- moved R24 96.4 mm to (116.8, 75.7), turned to 180 degrees
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Connections:
- IC1 pad 25: /DAC/SPDIF2 -> /DAC/SPDIF1
- IC1 pad 27: /DAC/SPDIF1 -> /DAC/SPDIF2
- IC3 pad 6: /DAC/AMP_SGND -> GNDA
- J6 pad S: /DAC/AMP_SGND -> GNDA
- U2 pad 5: unconnected-(U2-EN-Pad5) -> Net-(U2-EN)
Routing:
- net /Buck/VOUT: track 25.9 -> 61.9 mm, vias 2 -> 3
- net /DAC/OUT_SE_L: track 7.28 -> 43.1 mm
- net /DAC/OUT_SE_R: track 8.38 -> 44.1 mm
- net Net-(D1-K): track 39.8 -> 4.25 mm
- net /UINN: track 4.10 -> 27.9 mm, vias 0 -> 1
- net /UINP: track 5.08 -> 27.1 mm, vias 0 -> 1
- net /SAMD11/USB.DN: track 20.0 -> 0.00 mm, vias 1 -> 0
- net /SAMD11/USB.DP: track 19.7 -> 0.00 mm, vias 1 -> 0
- net SWITCH_LOW: track 15.1 -> 33.8 mm
- net /DAC/SPDIF1: track 1.85 -> 20.3 mm
- net Net-(J6-PadR): track 17.3 -> 3.27 mm
- net VBUS: track 30.8 -> 17.1 mm, vias 2 -> 0
- net Net-(IC1-ADDR): track 1.93 -> 14.3 mm, vias 1 -> 2
- net /DAC/OUT_BAL.R+: track 0.00 -> 12.2 mm
- net /DAC/OUT_BAL.R-: track 0.00 -> 12.0 mm, vias 0 -> 2
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- added copper zone on B.Cu, net Net-(U2-SW)
Other:
- board size 175.3 x 50.1 mm -> 148.4 x 50.1 mm
