File: d-lev-io/buck.kicad_sch (KiCad schematic)
At the start: 14 parts, among them U3 TPS54202DDC

Commit message: Add footprint references and fix error in buck schematic
Parts:
- C16: footprint (none) -> Capacitor_SMD:C_0805_2012Metric
- C17: footprint (none) -> Capacitor_SMD:C_1210_3225Metric; Voltage 30V 2A -> 30V 2A X5R
- C20: footprint (none) -> Resistor_SMD:R_0805_2012Metric
- C21: footprint (none) -> Capacitor_SMD:C_0603_1608Metric
- C23, C24: footprint (none) -> Capacitor_SMD:C_1210_3225Metric
- L1: footprint (none) -> Inductor_SMD:L_Bourns_SRN8040TA
- R19: footprint (none) -> Resistor_SMD:R_0603_1608Metric
Connections:
- net VIN: now also R18.2, U3.3 (VIN); no longer JP2.2 (B), R18.1, U3.5 (EN)
- new net: JP2.2 (B), R18.1, U3.5 (EN)
Other:
- moved on the sheet: JP2, L1, R18, R19

Commit message: many more changes
Parts:
- JP2: footprint (none) -> Jumper:SolderJumper-2_P1.3mm_Bridged_RoundedPad1.0x1.5mm
- R11: renamed from R18; footprint (none) -> Resistor_SMD:R_0805_2012Metric
- R12: renamed from R19; footprint Resistor_SMD:R_0603_1608Metric -> Resistor_SMD:R_0805_2012Metric
- R13: renamed from R17; footprint (none) -> Resistor_SMD:R_0805_2012Metric
- R14: renamed from R15; footprint (none) -> Resistor_SMD:R_0805_2012Metric
- R15: renamed from R16; footprint (none) -> Resistor_SMD:R_0805_2012Metric
- renumbered C17 to C13, C16 to C14, C20 to C15, C21 to C16, C23 to C17, C24 to C18

Commit message: map SAMD21 pins
Parts:
- C14: value 0.1u -> .1u
- C15: value 0.1u -> .1u; footprint Resistor_SMD:R_0805_2012Metric -> Capacitor_SMD:C_0805_2012Metric
Changed lines of the file:
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@@
       (effects (font (size 1.27 1.27)) (justify left))
     )
-    (property "Value" "0.1u" (at 107.95 93.345 0)
+    (property "Value" ".1u" (at 107.95 93.345 0)
       (effects (font (size 1.27 1.27)) (justify left))
     )
@@
       (effects (font (size 1.27 1.27)))
     )
-    (property "Value" "0.1u" (at 168.91 78.74 90)
+    (property "Value" ".1u" (at 168.91 78.74 90)
       (effects (font (size 1.27 1.27)))
     )
-    (property "Footprint" "Resistor_SMD:R_0805_2012Metric" (at 172.72 81.5848 0)
+    (property "Footprint" "Capacitor_SMD:C_0805_2012Metric" (at 172.72 81.5848 0)
       (effects (font (size 1.27 1.27)) hide)
     )

Commit message: many board updates
Parts:
- removed JP2: BUCK_VERSION, Jumper:SolderJumper-2_P1.3mm_Bridged_RoundedPad1.0x1.5mm, symbol Jumper:Jumper_2_Bridged
- removed R11: 510k, Resistor_SMD:R_0805_2012Metric, symbol Device:R_Small
- removed R12: 105k, Resistor_SMD:R_0805_2012Metric, symbol Device:R_Small
Connections:
- no-connect marks 0 -> 1
Other:
- note added: "In 12-28V"
- note added: "Out 5V@1A"
- note added: "Remove R42 if using 54202H"
- note removed: "Cut jumper if using 54202H"
Changed lines of the file:
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@@
 (kicad_sch (version 20230121) (generator eeschema)
   (paper "A4")
-  (junction (at 131.445 90.17) (diameter 0) (color 0 0 0 0)
-  )
   (junction (at 172.72 85.09) (diameter 0) (color 0 0 0 0)
   )
@@
   (junction (at 104.14 82.55) (diameter 0) (color 0 0 0 0)
   )
-  (junction (at 131.445 82.55) (diameter 0) (color 0 0 0 0)
-  )
   (junction (at 207.01 85.09) (diameter 0) (color 0 0 0 0)
   )
   (junction (at 193.675 106.68) (diameter 0) (color 0 0 0 0)
   )
+  (no_connect (at 144.78 87.63))
   (wire (pts (xy 171.45 82.55) (xy 172.72 82.55))
     (stroke (width 0) (type default))
@@
     (stroke (width 0) (type default))
   )
-  (wire (pts (xy 131.445 88.9) (xy 131.445 90.17))
-    (stroke (width 0) (type default))
-  )
   (wire (pts (xy 217.17 85.09) (xy 223.52 85.09))
     (stroke (width 0) (type default))
@@
     (stroke (width 0) (type default))
   )
-  (wire (pts (xy 104.14 82.55) (xy 131.445 82.55))
+  (wire (pts (xy 104.14 82.55) (xy 144.78 82.55))
     (stroke (width 0) (type default))
   )
@@
     (stroke (width 0) (type default))
   )
-  (wire (pts (xy 131.445 83.82) (xy 131.445 82.55))
-    (stroke (width 0) (type default))
-  )
   (wire (pts (xy 217.17 92.71) (xy 217.17 95.25))
     (stroke (width 0) (type default))
@@
     (stroke (width 0) (type default))
   )
-  (wire (pts (xy 131.445 82.55) (xy 144.78 82.55))
-    (stroke (width 0) (type default))
-  )
-  (wire (pts (xy 131.445 109.855) (xy 131.445 112.395))
-    (stroke (width 0) (type default))
-  )
   (wire (pts (xy 91.44 93.98) (xy 91.44 101.6))
     (stroke (width 0) (type default))
@@
     (stroke (width 0) (type default))
   )
-  (wire (pts (xy 131.445 90.17) (xy 131.445 92.075))
-    (stroke (width 0) (type default))
-  )
   (wire (pts (xy 179.07 106.68) (xy 184.785 106.68))
     (stroke (width 0) (type default))
   )
-  (wire (pts (xy 144.78 90.17) (xy 131.445 90.17))
-    (stroke (width 0) (type default))
-  )
-  (wire (pts (xy 144.78 87.63) (xy 144.78 90.17))
-    (stroke (width 0) (type default))
-  )
   (wire (pts (xy 166.37 82.55) (xy 165.1 82.55))
     (stroke (width 0) (type default))
@@
   )
   (wire (pts (xy 212.09 95.25) (xy 212.09 97.79))
-    (stroke (width 0) (type default))
-  )
-  (wire (pts (xy 131.445 104.775) (xy 131.445 102.235))
     (stroke (width 0) (type default))
   )
@@
     (effects (font (size 1.27 1.27)) (justify left bottom))
   )
+  (text "In 12-28V" (at 83.439 79.883 0)
+    (effects (font (size 1.27 1.27)) (justify left bottom))
+  )
   (text "Use Murata tool to find capacitors with lowest ESR at switching frequency for a given buck converter:\nhttps://ds.murata.co.jp/simsurfing/mlcc.html?lcid=en-us&jis=false&md5=af9fcec8873ac9edcee66de8ca92af94\nESR vs frequency depends more on case size than capacitance value\nUse two capacitors in parallel to drop ESR (one higher C, one lower C) to cover lower-ESR spectrum\n-> big, high capacitance, little, lower capacitance"
     (at 159.385 30.48 0)
@@
     (effects (font (size 1.27 1.27)) (justify left bottom))
   )
-  (text "Cut jumper if using 54202H" (at 123.825 88.265 90)
+  (text "Out 5V@1A" (at 216.916 82.042 0)
+    (effects (font (size 1.27 1.27)) (justify left bottom))
+  )
+  (text "Remove R42 if using 54202H" (at 123.825 88.265 90)
     (effects (font (size 1.27 1.27)) (justify right bottom))
   )
@@
     )
   )
-  (symbol (lib_id "Device:R_Small") (at 131.445 107.315 0) (unit 1)
-    (in_bom yes) (on_board yes) (dnp no) (fields_autoplaced)
-    (property "Reference" "R12" (at 133.985 106.68 0)
-      (effects (font (size 1.27 1.27)) (justify left))
-    )
-    (property "Value" "105k" (at 133.985 109.22 0)
-      (effects (font (size 1.27 1.27)) (justify left))
-    )
-    (property "Footprint" "Resistor_SMD:R_0805_2012Metric" (at 129.667 107.315 90)
-      (effects (font (size 1.27 1.27)) hide)
-    )
-    (property "Datasheet" "~" (at 131.445 107.315 0)
-      (effects (font (size 1.27 1.27)) hide)
-    )
-    (property "Tolerance" "1%" (at 131.445 107.315 0)
-      (effects (font (size 1.27 1.27)) hide)
-    )
-    (pin "1")
-    (pin "2")
-    (instances
-      (project "d-lev-io"
-        (path "/9261a07b-ae4a-4d72-8042-ea097cd0e5ed/f19ba83a-ef5a-459f-9ba4-5cb53e267077"
-          (reference "R12") (unit 1)
-        )
-      )
-    )
-  )
   (symbol (lib_id "Device:C_Small") (at 91.44 91.44 0) (unit 1)
     (in_bom yes) (on_board yes) (dnp no) (fields_autoplaced)
@@
     )
   )
-  (symbol (lib_id "Jumper:Jumper_2_Bridged") (at 131.445 97.155 90) (unit 1)
-    (in_bom yes) (on_board yes) (dnp no)
-    (property "Reference" "JP2" (at 126.365 97.155 0)
-      (effects (font (size 1.27 1.27)))
-    )
-    (property "Value" "BUCK_VERSION" (at 128.905 97.155 0)
-      (effects (font (size 1.27 1.27)))
-    )
-    (property "Footprint" "Jumper:SolderJumper-2_P1.3mm_Bridged_RoundedPad1.0x1.5mm" (at 131.445 97.155 0)
-      (effects (font (size 1.27 1.27)) hide)
-    )
-    (property "Datasheet" "~" (at 131.445 97.155 0)
-      (effects (font (size 1.27 1.27)) hide)
-    )
-    (pin "1")
-    (pin "2")
-    (instances
-      (project "d-lev-io"
-        (path "/9261a07b-ae4a-4d72-8042-ea097cd0e5ed/f19ba83a-ef5a-459f-9ba4-5cb53e267077"
-          (reference "JP2") (unit 1)
-        )
-      )
-    )
-  )
-  (symbol (lib_id "power:GND") (at 131.445 112.395 0) (unit 1)
-    (in_bom yes) (on_board yes) (dnp no) (fields_autoplaced)
-    (property "Reference" "#PWR031" (at 131.445 118.745 0)
-      (effects (font (size 1.27 1.27)) hide)
-    )
-    (property "Value" "GND" (at 131.445 117.475 0)
-      (effects (font (size 1.27 1.27)))
-    )
-    (property "Footprint" "" (at 131.445 112.395 0)
-      (effects (font (size 1.27 1.27)) hide)
-    )
-    (property "Datasheet" "" (at 131.445 112.395 0)
-      (effects (font (size 1.27 1.27)) hide)
-    )
-    (pin "1")
-    (instances
-      (project "d-lev-io"
-        (path "/9261a07b-ae4a-4d72-8042-ea097cd0e5ed/f19ba83a-ef5a-459f-9ba4-5cb53e267077"
-          (reference "#PWR031") (unit 1)
-        )
-      )
-    )
-  )
   (symbol (lib_id "Device:C_Small") (at 168.91 82.55 90) (unit 1)
     (in_bom yes) (on_board yes) (dnp no) (fields_autoplaced)
@@
         )
       )
-    )
-  )
-  (symbol (lib_id "Device:R_Small") (at 131.445 86.36 180) (unit 1)
-    (in_bom yes) (on_board yes) (dnp no) (fields_autoplaced)
-    (property "Reference" "R11" (at 133.985 85.725 0)
-      (effects (font (size 1.27 1.27)) (justify right))
-    )
-    (property "Value" "510k" (at 133.985 88.265 0)
-      (effects (font (size 1.27 1.27)) (justify right))
-    )
-    (property "Footprint" "Resistor_SMD:R_0805_2012Metric" (at 133.223 86.36 90)
-      (effects (font (size 1.27 1.27)) hide)
-    )
-    (property "Datasheet" "~" (at 131.445 86.36 0)
-      (effects (font (size 1.27 1.27)) hide)
-    )
-    (property "Tolerance" "1%" (at 131.445 86.36 0)
-      (effects (font (size 1.27 1.27)) hide)
-    )
-    (pin "1")
-    (pin "2")
-    (instances
-      (project "d-lev-io"
-        (path "/9261a07b-ae4a-4d72-8042-ea097cd0e5ed/f19ba83a-ef5a-459f-9ba4-5cb53e267077"
-          (reference "R11") (unit 1)
-        )
-      )

Commit message: more routing
Parts:
- added R11: 511k, Resistor_SMD:R_0603_1608Metric, symbol Device:R_Small
- added R12: 105k, Resistor_SMD:R_0603_1608Metric, symbol Device:R_Small
Connections:
- net GND: now also R12.2
- net at U3.5 (EN): now also R11.1
- new net: R11.2, R12.1
- no-connect marks 1 -> 0
Changed lines of the file:
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@@
   (junction (at 193.675 106.68) (diameter 0) (color 0 0 0 0)
   )
-  (no_connect (at 144.78 87.63))
   (wire (pts (xy 171.45 82.55) (xy 172.72 82.55))
     (stroke (width 0) (type default))
@@
     (stroke (width 0) (type default))
   )
+  (wire (pts (xy 137.795 98.806) (xy 137.795 95.25))
+    (stroke (width 0) (type default))
+  )
   (wire (pts (xy 193.675 93.98) (xy 193.675 97.79))
     (stroke (width 0) (type default))
@@
     (stroke (width 0) (type default))
   )
+  (wire (pts (xy 137.795 90.17) (xy 137.795 87.63))
+    (stroke (width 0) (type default))
+  )
+  (wire (pts (xy 137.795 106.426) (xy 137.795 103.886))
+    (stroke (width 0) (type default))
+  )
   (wire (pts (xy 91.44 82.55) (xy 83.82 82.55))
+    (stroke (width 0) (type default))
+  )
+  (wire (pts (xy 137.795 87.63) (xy 144.78 87.63))
     (stroke (width 0) (type default))
   )
@@
         (path "/9261a07b-ae4a-4d72-8042-ea097cd0e5ed/f19ba83a-ef5a-459f-9ba4-5cb53e267077"
           (reference "C17") (unit 1)
+        )
+      )
+    )
+  )
+  (symbol (lib_id "Device:R_Small") (at 137.795 101.346 0) (unit 1)
+    (in_bom yes) (on_board yes) (dnp no) (fields_autoplaced)
+    (property "Reference" "R12" (at 139.9032 100.711 0)
+      (effects (font (size 1.27 1.27)) (justify left))
+    )
+    (property "Value" "105k" (at 139.9032 103.251 0)
+      (effects (font (size 1.27 1.27)) (justify left))
+    )
+    (property "Footprint" "Resistor_SMD:R_0603_1608Metric" (at 136.017 101.346 90)
+      (effects (font (size 1.27 1.27)) hide)
+    )
+    (property "Datasheet" "~" (at 137.795 101.346 0)
+      (effects (font (size 1.27 1.27)) hide)
+    )
+    (property "Tolerance" "1%" (at 137.795 101.346 0)
+      (effects (font (size 1.27 1.27)) hide)
+    )
+    (pin "1")
+    (pin "2")
+    (instances
+      (project "d-lev-io"
+        (path "/9261a07b-ae4a-4d72-8042-ea097cd0e5ed/f19ba83a-ef5a-459f-9ba4-5cb53e267077"
+          (reference "R12") (unit 1)
         )
       )
@@
         )
       )
+    )
+  )
+  (symbol (lib_id "power:GND") (at 137.795 106.426 0) (unit 1)
+    (in_bom yes) (on_board yes) (dnp no) (fields_autoplaced)
+    (property "Reference" "#PWR081" (at 137.795 112.776 0)
+      (effects (font (size 1.27 1.27)) hide)
+    )
+    (property "Value" "GND" (at 137.795 111.506 0)
+      (effects (font (size 1.27 1.27)))
+    )
+    (property "Footprint" "" (at 137.795 106.426 0)
+      (effects (font (size 1.27 1.27)) hide)
+    )
+    (property "Datasheet" "" (at 137.795 106.426 0)
+      (effects (font (size 1.27 1.27)) hide)
+    )
+    (pin "1")
+    (instances
+      (project "d-lev-io"
+        (path "/9261a07b-ae4a-4d72-8042-ea097cd0e5ed/f19ba83a-ef5a-459f-9ba4-5cb53e267077"
+          (reference "#PWR081") (unit 1)
+        )
+      )
+    )
+  )
+  (symbol (lib_id "Device:R_Small") (at 137.795 92.71 0) (unit 1)
+    (in_bom yes) (on_board yes) (dnp no) (fields_autoplaced)
+    (property "Reference" "R11" (at 140.335 92.075 0)
+      (effects (font (size 1.27 1.27)) (justify left))
+    )
+    (property "Value" "511k" (at 140.335 94.615 0)
+      (effects (font (size 1.27 1.27)) (justify left))
+    )
+    (property "Footprint" "Resistor_SMD:R_0603_1608Metric" (at 136.017 92.71 90)
+      (effects (font (size 1.27 1.27)) hide)
+    )
+    (property "Datasheet" "~" (at 137.795 92.71 0)
+      (effects (font (size 1.27 1.27)) hide)
+    )
+    (property "Tolerance" "1%" (at 137.795 92.71 0)
+      (effects (font (size 1.27 1.27)) hide)
+    )
+    (pin "1")
+    (pin "2")
+    (instances
+      (project "d-lev-io"
+        (path "/9261a07b-ae4a-4d72-8042-ea097cd0e5ed/f19ba83a-ef5a-459f-9ba4-5cb53e267077"
+          (reference "R11") (unit 1)
+        )
+      )
