File: d-lev-io/LDO.kicad_sch (KiCad schematic)
At the start: 6 parts, among them U5 AP2112K-3.3

Commit message: I/O board silk placement
Parts:
- renumbered U5 to U4
Changed lines of the file:
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@@
         )
         (path "/9261a07b-ae4a-4d72-8042-ea097cd0e5ed/83e88c30-a90d-4699-98a4-5fb5b0c65049"
-          (reference "C24") (unit 1)
+          (reference "C31") (unit 1)
         )
       )
@@
         )
         (path "/9261a07b-ae4a-4d72-8042-ea097cd0e5ed/83e88c30-a90d-4699-98a4-5fb5b0c65049"
-          (reference "C27") (unit 1)
+          (reference "C21") (unit 1)
         )
       )
@@
         )
         (path "/9261a07b-ae4a-4d72-8042-ea097cd0e5ed/83e88c30-a90d-4699-98a4-5fb5b0c65049"
-          (reference "C26") (unit 1)
+          (reference "C23") (unit 1)
         )
       )
@@
         )
         (path "/9261a07b-ae4a-4d72-8042-ea097cd0e5ed/83e88c30-a90d-4699-98a4-5fb5b0c65049"
-          (reference "C23") (unit 1)
+          (reference "C26") (unit 1)
         )
       )
@@
   (symbol (lib_id "Regulator_Linear:AP2112K-3.3") (at 118.11 86.36 0) (unit 1)
     (in_bom yes) (on_board yes) (dnp no) (fields_autoplaced)
-    (property "Reference" "U5" (at 118.11 78.105 0)
+    (property "Reference" "U4" (at 118.11 78.105 0)
       (effects (font (size 1.27 1.27)))
     )
@@
       (project "d-lev-io"
         (path "/9261a07b-ae4a-4d72-8042-ea097cd0e5ed/83e88c30-a90d-4699-98a4-5fb5b0c65049"
-          (reference "U5") (unit 1)
+          (reference "U4") (unit 1)
         )
       )
