File: d-lev-io/LDO.kicad_sch (KiCad schematic)
At the start: 6 parts, among them U4 AP2112K-3.3

Commit message: Add iBOMs and additional part numbers
Parts:
- C12, C14: MPN (none) -> CL10B105KP8NNNC; Notes (none) -> Common; Supplier (none) -> Digi-Key; Supplier URL (none) -> https://www.digikey.com/en/products/detail/samsung-electro-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
- C13: MPN (none) -> CL21A106KAYNNNG; Notes (none) -> Common; Supplier (none) -> Mouser; Supplier Alt URL (none) -> https://www.mouser.com/ProductDetail/187-CL21A106KAYNNNG; Supplier URL (none) -> https://www.mouser.com/ProductDetail/187-CL21A106KAYNNNG
- C15: value .1u -> 100n; MPN (none) -> GRM188R71E104KA01D; Notes (none) -> Common; Supplier (none) -> Digi-Key; Supplier URL (none) -> https://www.digikey.com/en/products/detail/murata-electroni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
- U4: MPN (none) -> AP2112K-3.3TRG1; Supplier (none) -> Mouser; Supplier URL (none) -> https://www.mouser.com/ProductDetail/621-AP2112K-3.3TRG1
Changed lines of the file:
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@@
       (effects (font (size 1.27 1.27)) hide)
     )
-    (property "Datasheet" "~" (at 140.335 91.44 0)
+    (property "Datasheet" "https://media.digikey.com/pdf/Data%20Sheets/Samsung%20PDFs/CL10B105KP8NNNC_Spec.pdf" (at 140.335 91.44 0)
+      (effects (font (size 1.27 1.27)) hide)
+    )
+    (property "Notes" "Common" (at 140.335 91.44 0)
+      (effects (font (size 1.27 1.27)) hide)
+    )
+    (property "Supplier Alt" "" (at 140.335 91.44 0)
+      (effects (font (size 1.27 1.27)) hide)
+    )
+    (property "Supplier Alt URL" "" (at 140.335 91.44 0)
+      (effects (font (size 1.27 1.27)) hide)
+    )
+    (property "Supplier URL" "https://www.digikey.com/en/products/detail/samsung-electro-mechanics/CL10B105KP8NNNC/3887604" (at 140.335 91.44 0)
+      (effects (font (size 1.27 1.27)) hide)
+    )
+    (property "DNP" "" (at 140.335 91.44 0)
+      (effects (font (size 1.27 1.27)) hide)
+    )
+    (property "MPN" "CL10B105KP8NNNC" (at 140.335 91.44 0)
+      (effects (font (size 1.27 1.27)) hide)
+    )
+    (property "Supplier" "Digi-Key" (at 140.335 91.44 0)
       (effects (font (size 1.27 1.27)) hide)
     )
@@
       (effects (font (size 1.27 1.27)) (justify right))
     )
-    (property "Value" ".1u" (at 153.67 93.3386 0)
+    (property "Value" "100n" (at 153.67 93.3386 0)
       (effects (font (size 1.27 1.27)) (justify right))
     )
@@
       (effects (font (size 1.27 1.27)) hide)
     )
-    (property "Datasheet" "~" (at 150.495 91.44 0)
+    (property "Datasheet" "https://search.murata.co.jp/Ceramy/image/img/A01X/G101/ENG/GRM188R71E104KA01-01.pdf" (at 150.495 91.44 0)
       (effects (font (size 1.27 1.27)) hide)
     )
@@
       (effects (font (size 1.27 1.27)))
     )
+    (property "Notes" "Common" (at 150.495 91.44 0)
+      (effects (font (size 1.27 1.27)) hide)
+    )
+    (property "Supplier Alt" "" (at 150.495 91.44 0)
+      (effects (font (size 1.27 1.27)) hide)
+    )
+    (property "Supplier Alt URL" "" (at 150.495 91.44 0)
+      (effects (font (size 1.27 1.27)) hide)
+    )
+    (property "Supplier URL" "https://www.digikey.com/en/products/detail/murata-electronics/GRM188R71E104KA01D/587154" (at 150.495 91.44 0)
+      (effects (font (size 1.27 1.27)) hide)
+    )
+    (property "Supplier" "Digi-Key" (at 150.495 91.44 0)
+      (effects (font (size 1.27 1.27)) hide)
+    )
+    (property "DNP" "" (at 150.495 91.44 0)
+      (effects (font (size 1.27 1.27)) hide)
+    )
+    (property "MPN" "GRM188R71E104KA01D" (at 150.495 91.44 0)
+      (effects (font (size 1.27 1.27)) hide)
+    )
     (pin "1")
     (pin "2")
@@
       (effects (font (size 1.27 1.27)) hide)
     )
-    (property "Datasheet" "~" (at 99.06 90.17 0)
+    (property "Datasheet" "https://media.digikey.com/pdf/Data%20Sheets/Samsung%20PDFs/CL10B105KP8NNNC_Spec.pdf" (at 99.06 90.17 0)
+      (effects (font (size 1.27 1.27)) hide)
+    )
+    (property "Notes" "Common" (at 99.06 90.17 0)
+      (effects (font (size 1.27 1.27)) hide)
+    )
+    (property "Supplier Alt" "" (at 99.06 90.17 0)
+      (effects (font (size 1.27 1.27)) hide)
+    )
+    (property "Supplier Alt URL" "" (at 99.06 90.17 0)
+      (effects (font (size 1.27 1.27)) hide)
+    )
+    (property "Supplier URL" "https://www.digikey.com/en/products/detail/samsung-electro-mechanics/CL10B105KP8NNNC/3887604" (at 99.06 90.17 0)
+      (effects (font (size 1.27 1.27)) hide)
+    )
+    (property "DNP" "" (at 99.06 90.17 0)
+      (effects (font (size 1.27 1.27)) hide)
+    )
+    (property "MPN" "CL10B105KP8NNNC" (at 99.06 90.17 0)
+      (effects (font (size 1.27 1.27)) hide)
+    )
+    (property "Supplier" "Digi-Key" (at 99.06 90.17 0)
       (effects (font (size 1.27 1.27)) hide)
     )
@@
       (effects (font (size 1.27 1.27)) hide)
     )
-    (property "Datasheet" "~" (at 89.535 90.17 0)
+    (property "Datasheet" "https://www.mouser.com/datasheet/2/585/MLCC-1837944.pdf" (at 89.535 90.17 0)
       (effects (font (size 1.27 1.27)) hide)
     )
@@
       (effects (font (size 1.27 1.27)))
     )
+    (property "Notes" "Common" (at 89.535 90.17 0)
+      (effects (font (size 1.27 1.27)) hide)
+    )
+    (property "Supplier Alt" "" (at 89.535 90.17 0)
+      (effects (font (size 1.27 1.27)) hide)
+    )
+    (property "Supplier Alt URL" "https://www.mouser.com/ProductDetail/187-CL21A106KAYNNNG" (at 89.535 90.17 0)
+      (effects (font (size 1.27 1.27)) hide)
+    )
+    (property "Supplier URL" "https://www.mouser.com/ProductDetail/187-CL21A106KAYNNNG" (at 89.535 90.17 0)
+      (effects (font (size 1.27 1.27)) hide)
+    )
+    (property "MPN" "CL21A106KAYNNNG" (at 89.535 90.17 0)
+      (effects (font (size 1.27 1.27)) hide)
+    )
+    (property "Supplier" "Mouser" (at 89.535 90.17 0)
+      (effects (font (size 1.27 1.27)) hide)
+    )
+    (property "DNP" "" (at 89.535 90.17 0)
+      (effects (font (size 1.27 1.27)) hide)
+    )
     (pin "1")
     (pin "2")
@@
       (effects (font (size 1.27 1.27)) hide)
     )
-    (property "Datasheet" "~" (at 130.81 91.44 0)
+    (property "Datasheet" "https://www.mouser.com/datasheet/2/585/MLCC-1837944.pdf" (at 130.81 91.44 0)
       (effects (font (size 1.27 1.27)) hide)
     )
@@
       (effects (font (size 1.27 1.27)))
     )
+    (property "Notes" "Common" (at 130.81 91.44 0)
+      (effects (font (size 1.27 1.27)) hide)
+    )
+    (property "Supplier Alt" "" (at 130.81 91.44 0)
+      (effects (font (size 1.27 1.27)) hide)
+    )
+    (property "Supplier Alt URL" "https://www.mouser.com/ProductDetail/187-CL21A106KAYNNNG" (at 130.81 91.44 0)
+      (effects (font (size 1.27 1.27)) hide)
+    )
+    (property "Supplier URL" "https://www.mouser.com/ProductDetail/187-CL21A106KAYNNNG" (at 130.81 91.44 0)
+      (effects (font (size 1.27 1.27)) hide)
+    )
+    (property "MPN" "CL21A106KAYNNNG" (at 130.81 91.44 0)
+      (effects (font (size 1.27 1.27)) hide)
+    )
+    (property "Supplier" "Mouser" (at 130.81 91.44 0)
+      (effects (font (size 1.27 1.27)) hide)
+    )
+    (property "DNP" "" (at 130.81 91.44 0)
+      (effects (font (size 1.27 1.27)) hide)
+    )
     (pin "1")
     (pin "2")
@@
       (effects (font (size 1.27 1.27)) hide)
     )
+    (property "Notes" "" (at 118.11 86.36 0)
+      (effects (font (size 1.27 1.27)) hide)
+    )
+    (property "Supplier Alt" "" (at 118.11 86.36 0)
+      (effects (font (size 1.27 1.27)) hide)
+    )
+    (property "Supplier Alt URL" "" (at 118.11 86.36 0)
+      (effects (font (size 1.27 1.27)) hide)
+    )
+    (property "Supplier URL" "https://www.mouser.com/ProductDetail/621-AP2112K-3.3TRG1" (at 118.11 86.36 0)
+      (effects (font (size 1.27 1.27)) hide)
+    )
+    (property "MPN" "AP2112K-3.3TRG1" (at 118.11 86.36 0)
+      (effects (font (size 1.27 1.27)) hide)
+    )
+    (property "Supplier" "Mouser" (at 118.11 86.36 0)
+      (effects (font (size 1.27 1.27)) hide)
+    )
+    (property "DNP" "" (at 118.11 86.36 0)
+      (effects (font (size 1.27 1.27)) hide)
+    )
