File: d-lev-afe/d-lev-afe.kicad_sch (KiCad schematic)
At the start: 29 parts, among them J1 S8B-PH-SM4-TB, Q1 MMBT3904, Q2 MMBT3906, U1 74AHC04, U2 HT7833-2, U3 SRV05-4

Commit message: pushed smaller AFE board
Parts:
- added H1, H2, H3, H4: MountingHole, MountingHole:MountingHole_3.2mm_M3, symbol Mechanical:MountingHole
- added H5: MountingHole_Pad, MountingHole:MountingHole_6.5mm_Pad_TopBottom, symbol Mechanical:MountingHole_Pad
Connections:
- net L_IN: now also H5.1
